File: is31se5100/is31se5100.sch (KiCad schematic (older format))
At the start: 1093 parts, among them J1 Conn_01x01, J10 Conn_01x05, J11 Conn_01x08, J12 Screw_Terminal_01x02, J13 Conn_01x08, J14 Conn_01x08, J15 Conn_01x08, J16 Conn_01x03, J17 Conn_01x01, J18 Conn_01x08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

Commit message: Established is31se5100_chained
Other:
- moved on the sheet: C1, C10, C11, C12, C13, C14, C15, C16, C17, C18, C19, C2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
