File: capacitive_fingerboard_guitar_650/capacitive_fingerboard_guitar_650.kicad_pcb (KiCad board)
At the start: 2 copper layers, 60.6 x 500 mm, 24 parts, among them J1 Conn_01x20, J2 Conn_01x20, J3 Conn_01x20, J4 Conn_01x20, U1 Electrode, U10 Electrode, U11 Electrode, U12 Electrode, U13 Electrode, U14 Electrode, U15 Electrode, U16 Electrode, U17 Electrode, U18 Electrode, U19 Electrode, U2 Electrode, U20 Electrode, U3 Electrode, U4 Electrode, U5 Electrode, U6 Electrode, U7 Electrode, U8 Electrode, U9 Electrode

Commit message: Added frets on E2 string
Parts:
- added J2: Conn_01x20, Connector_PinHeader_2.54mm:PinHeader_1x20_P2.54mm_Vertical, F.Cu at (-326.9, 398.4)
- added J3: Conn_01x20, Connector_PinHeader_2.54mm:PinHeader_1x20_P2.54mm_Vertical, F.Cu at (-345.4, 398.4)
- added J4: Conn_01x20, Connector_PinHeader_2.54mm:PinHeader_1x20_P2.54mm_Vertical, F.Cu at (-340.8, 398.4)
- added J5: Conn_01x20, Connector_PinHeader_2.54mm:PinHeader_1x20_P2.54mm_Vertical, F.Cu at (-336.1, 398.4)
- added J6: Conn_01x20, Connector_PinHeader_2.54mm:PinHeader_1x20_P2.54mm_Vertical, F.Cu at (-2.50, 505.6)
- added U100: Electrode, Custom_Electrode:Circle_2mm, F.Cu at (-290.9, 411.7)
- added U101: Electrode, Custom_Electrode:Circle_2mm, F.Cu at (-299.2, 416.6)
- added U102: Electrode, Custom_Electrode:Circle_2mm, F.Cu at (-296.2, 416.6)
- added U103: Electrode, Custom_Electrode:Circle_2mm, F.Cu at (-302.2, 421.6)
- added U104: Electrode, Custom_Electrode:Circle_2mm, F.Cu at (-308.2, 426.5)
- added U105: Electrode, Custom_Electrode:Circle_2mm, F.Cu at (-305.2, 426.5)
- added U106: Electrode, Custom_Electrode:Circle_2mm, F.Cu at (-314.2, 431.5)
- added U107: Electrode, Custom_Electrode:Circle_2mm, F.Cu at (-311.2, 431.5)
- added U108: Electrode, Custom_Electrode:Circle_2mm, F.Cu at (-302.2, 426.5)
- added U109: Electrode, Custom_Electrode:Circle_2mm, F.Cu at (-323.2, 441.4)
- added U110: Electrode, Custom_Electrode:Circle_2mm, F.Cu at (-320.2, 441.4)
- added U111: Electrode, Custom_Electrode:Circle_2mm, F.Cu at (-278.9, 401.8)
- added U112: Electrode, Custom_Electrode:Circle_2mm, F.Cu at (-314.2, 436.4)
- added U113: Electrode, Custom_Electrode:Circle_2mm, F.Cu at (-299.2, 421.6)
- added U114: Electrode, Custom_Electrode:Circle_2mm, F.Cu at (-275.9, 401.8)
- added U115: Electrode, Custom_Electrode:Circle_2mm, F.Cu at (-296.2, 421.6)
- added U116: Electrode, Custom_Electrode:Circle_2mm, F.Cu at (-311.2, 436.4)
- added U117: Electrode, Custom_Electrode:Circle_2mm, F.Cu at (-317.2, 441.4)
- added U118: Electrode, Custom_Electrode:Circle_2mm, F.Cu at (-323.2, 446.3)
- added U119: Electrode, Custom_Electrode:Circle_2mm, F.Cu at (-308.2, 431.5)
- added U120: Electrode, Custom_Electrode:E4_Fret20, F.Cu at (47.0, 430.1)
- added U21: Electrode, Custom_Electrode:Circle_2mm, F.Cu at (-317.9, 396.8)
- added U22: Electrode, Custom_Electrode:Circle_2mm, F.Cu at (-314.9, 396.8)
- added U23: Electrode, Custom_Electrode:Circle_2mm, F.Cu at (-311.9, 396.8)
- added U24: Electrode, Custom_Electrode:Circle_2mm, F.Cu at (-308.9, 396.8)
- added U25: Electrode, Custom_Electrode:Circle_2mm, F.Cu at (-305.9, 396.8)
- added U26: Electrode, Custom_Electrode:Circle_2mm, F.Cu at (-302.9, 396.8)
- added U27: Electrode, Custom_Electrode:Circle_2mm, F.Cu at (-299.9, 396.8)
- added U28: Electrode, Custom_Electrode:Circle_2mm, F.Cu at (-296.9, 396.8)
- added U29: Electrode, Custom_Electrode:Circle_2mm, F.Cu at (-317.2, 436.4)
- added U30: Electrode, Custom_Electrode:Circle_2mm, F.Cu at (-320.9, 401.8)
- added U31: Electrode, Custom_Electrode:Circle_2mm, F.Cu at (-317.9, 401.8)
- added U32: Electrode, Custom_Electrode:Circle_2mm, F.Cu at (-314.9, 401.8)
- added U33: Electrode, Custom_Electrode:Circle_2mm, F.Cu at (-311.9, 401.8)
- added U34: Electrode, Custom_Electrode:Circle_2mm, F.Cu at (-308.9, 401.8)
- added U35: Electrode, Custom_Electrode:Circle_2mm, F.Cu at (-305.9, 401.8)
- added U36: Electrode, Custom_Electrode:Circle_2mm, F.Cu at (-302.9, 401.8)
- added U37: Electrode, Custom_Electrode:Circle_2mm, F.Cu at (-299.9, 401.8)
- added U38: Electrode, Custom_Electrode:Circle_2mm, F.Cu at (-320.9, 406.7)
- added U39: Electrode, Custom_Electrode:Circle_2mm, F.Cu at (-317.9, 406.7)
- added U40: Electrode, Custom_Electrode:Circle_2mm, F.Cu at (-314.9, 406.7)
- added U41: Electrode, Custom_Electrode:Circle_2mm, F.Cu at (-311.9, 406.7)
- added U42: Electrode, Custom_Electrode:Circle_2mm, F.Cu at (-320.9, 396.8)
- added U43: Electrode, Custom_Electrode:Circle_2mm, F.Cu at (-305.9, 406.7)
- added U44: Electrode, Custom_Electrode:Circle_2mm, F.Cu at (-320.9, 411.7)
- added U45: Electrode, Custom_Electrode:Circle_2mm, F.Cu at (-317.9, 411.7)
- added U46: Electrode, Custom_Electrode:Circle_2mm, F.Cu at (-314.9, 411.7)
- added U47: Electrode, Custom_Electrode:Circle_2mm, F.Cu at (-311.9, 411.7)
- added U48: Electrode, Custom_Electrode:Circle_2mm, F.Cu at (-308.9, 411.7)
- added U49: Electrode, Custom_Electrode:Circle_2mm, F.Cu at (-323.2, 416.6)
- added U50: Electrode, Custom_Electrode:Circle_2mm, F.Cu at (-320.2, 416.6)
- added U51: Electrode, Custom_Electrode:Circle_2mm, F.Cu at (-317.2, 416.6)
- added U52: Electrode, Custom_Electrode:Circle_2mm, F.Cu at (-314.2, 416.6)
- added U53: Electrode, Custom_Electrode:Circle_2mm, F.Cu at (-323.2, 421.6)
- added U54: Electrode, Custom_Electrode:Circle_2mm, F.Cu at (-320.2, 421.6)
- added U55: Electrode, Custom_Electrode:Circle_2mm, F.Cu at (-293.9, 396.8)
- added U56: Electrode, Custom_Electrode:Circle_2mm, F.Cu at (-308.9, 406.7)
- added U57: Electrode, Custom_Electrode:Circle_2mm, F.Cu at (-314.2, 421.6)
- added U58: Electrode, Custom_Electrode:Circle_2mm, F.Cu at (-323.2, 426.5)
- added U59: Electrode, Custom_Electrode:Circle_2mm, F.Cu at (-320.2, 426.5)
- added U60: Electrode, Custom_Electrode:Circle_2mm, F.Cu at (-311.2, 416.6)
- added U61: Electrode, Custom_Electrode:Circle_2mm, F.Cu at (-305.9, 411.7)
- added U62: Electrode, Custom_Electrode:Circle_2mm, F.Cu at (-302.9, 406.7)
- added U63: Electrode, Custom_Electrode:Circle_2mm, F.Cu at (-299.9, 406.7)
- added U64: Electrode, Custom_Electrode:Circle_2mm, F.Cu at (-296.9, 401.8)
- added U65: Electrode, Custom_Electrode:Circle_2mm, F.Cu at (-293.9, 401.8)
- added U66: Electrode, Custom_Electrode:Circle_2mm, F.Cu at (-290.9, 396.8)
- added U67: Electrode, Custom_Electrode:Circle_2mm, F.Cu at (-287.9, 396.8)
- added U68: Electrode, Custom_Electrode:Circle_2mm, F.Cu at (-275.9, 396.8)
- added U69: Electrode, Custom_Electrode:Circle_2mm, F.Cu at (-323.2, 436.4)
- added U70: Electrode, Custom_Electrode:Circle_2mm, F.Cu at (-290.9, 401.8)
- added U71: Electrode, Custom_Electrode:Circle_2mm, F.Cu at (-296.9, 406.7)
- added U72: Electrode, Custom_Electrode:Circle_2mm, F.Cu at (-302.9, 411.7)
- added U73: Electrode, Custom_Electrode:Circle_2mm, F.Cu at (-299.9, 411.7)
- added U74: Electrode, Custom_Electrode:Circle_2mm, F.Cu at (-308.2, 416.6)
- added U75: Electrode, Custom_Electrode:Circle_2mm, F.Cu at (-305.2, 416.6)
- added U76: Electrode, Custom_Electrode:Circle_2mm, F.Cu at (-311.2, 421.6)
- added U77: Electrode, Custom_Electrode:Circle_2mm, F.Cu at (-317.2, 426.5)
- added U78: Electrode, Custom_Electrode:Circle_2mm, F.Cu at (-314.2, 426.5)
- added U79: Electrode, Custom_Electrode:Circle_2mm, F.Cu at (-323.2, 431.5)
- added U80: Electrode, Custom_Electrode:Circle_2mm, F.Cu at (-320.2, 431.5)
- added U81: Electrode, Custom_Electrode:Circle_2mm, F.Cu at (-281.9, 401.8)
- added U82: Electrode, Custom_Electrode:Circle_2mm, F.Cu at (-284.9, 396.8)
- added U83: Electrode, Custom_Electrode:Circle_2mm, F.Cu at (-320.2, 436.4)
- added U84: Electrode, Custom_Electrode:Circle_2mm, F.Cu at (-311.2, 426.5)
- added U85: Electrode, Custom_Electrode:Circle_2mm, F.Cu at (-308.2, 421.6)
- added U86: Electrode, Custom_Electrode:Circle_2mm, F.Cu at (-305.2, 421.6)
- added U87: Electrode, Custom_Electrode:Circle_2mm, F.Cu at (-302.2, 416.6)
- added U88: Electrode, Custom_Electrode:Circle_2mm, F.Cu at (-296.9, 411.7)
- added U89: Electrode, Custom_Electrode:Circle_2mm, F.Cu at (-293.9, 406.7)
- added U90: Electrode, Custom_Electrode:Circle_2mm, F.Cu at (-290.9, 406.7)
- added U91: Electrode, Custom_Electrode:Circle_2mm, F.Cu at (-287.9, 401.8)
- added U92: Electrode, Custom_Electrode:Circle_2mm, F.Cu at (-284.9, 401.8)
- added U93: Electrode, Custom_Electrode:Circle_2mm, F.Cu at (-281.9, 396.8)
- added U94: Electrode, Custom_Electrode:Circle_2mm, F.Cu at (-278.9, 396.8)
- added U95: Electrode, Custom_Electrode:Circle_2mm, F.Cu at (-317.2, 431.5)
- added U96: Electrode, Custom_Electrode:Circle_2mm, F.Cu at (-317.2, 421.6)
- added U97: Electrode, Custom_Electrode:Circle_2mm, F.Cu at (-287.9, 406.7)
- added U98: Electrode, Custom_Electrode:Circle_2mm, F.Cu at (-284.9, 406.7)
- added U99: Electrode, Custom_Electrode:Circle_2mm, F.Cu at (-293.9, 411.7)
- U1: footprint Custom_Electrode:String_1.1684x36.482mm -> Custom_Electrode:E2_F2
- U10: footprint Custom_Electrode:Circle_2mm -> Custom_Electrode:E2_D3
- U11: footprint Custom_Electrode:Circle_2mm -> Custom_Electrode:E2_D#3
- U12: footprint Custom_Electrode:Circle_2mm -> Custom_Electrode:E2_E3
- U13: footprint Custom_Electrode:Circle_2mm -> Custom_Electrode:E2_F3
- U14: footprint Custom_Electrode:Circle_2mm -> Custom_Electrode:E2_F#3
- U15: footprint Custom_Electrode:Circle_2mm -> Custom_Electrode:E2_G3
- U16: footprint Custom_Electrode:Circle_2mm -> Custom_Electrode:E2_G#3
- U17: footprint Custom_Electrode:Circle_2mm -> Custom_Electrode:E2_A3
- U18: footprint Custom_Electrode:Circle_2mm -> Custom_Electrode:E2_A#3
- U19: footprint Custom_Electrode:Circle_2mm -> Custom_Electrode:E2_B3
- U2: footprint Custom_Electrode:String_1.1684x34.434mm -> Custom_Electrode:E2_F#2
- U20: footprint Custom_Electrode:Circle_2mm -> Custom_Electrode:E2_C4
- U3: footprint Custom_Electrode:Circle_2mm -> Custom_Electrode:E2_G2
- U4: footprint Custom_Electrode:Circle_2mm -> Custom_Electrode:E2_G#2
- U5: footprint Custom_Electrode:Circle_2mm -> Custom_Electrode:E2_A2
- U6: footprint Custom_Electrode:Circle_2mm -> Custom_Electrode:E2_A#2
- U7: footprint Custom_Electrode:Circle_2mm -> Custom_Electrode:E2_B2
- U8: footprint Custom_Electrode:Circle_2mm -> Custom_Electrode:E2_C3
- U9: footprint Custom_Electrode:Circle_2mm -> Custom_Electrode:E2_C#3
- moved U19 355.4 mm to (-9.95, 419.7)
- moved U18 347.0 mm to (-9.90, 406.6)
- moved U17 337.1 mm to (-10.2, 392.0)
- moved U16 312.4 mm to (-9.80, 376.1)
- moved U15 301.1 mm to (-10.2, 360.1)
- moved U14 287.6 mm to (-10.2, 341.9)
- moved U13 260.8 mm to (-9.95, 323.4)
- moved U12 252.7 mm to (-9.90, 304.1)
- moved U11 222.8 mm to (-9.50, 284.0)
- moved U10 209.6 mm to (-9.30, 262.4)
- moved U9 187.7 mm to (-9.60, 239.5)
- moved U8 160.5 mm to (-9.60, 215.7)
- moved U7 138.1 mm to (-9.25, 190.9)
- moved U6 115.4 mm to (-9.60, 162.8)
- moved J2 108.6 mm to (-110.5, 381.1)
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
Commit message: Added more frets on pcb
Parts:
- removed the J2 at (-110.5, 381.1)
- removed the J3 at (-109.5, 407.9)
- removed the J4 at (-1.75, 489.4)
- U21: footprint Custom_Electrode:Circle_2mm -> Custom_Electrode:A2_A#2
- U22: footprint Custom_Electrode:Circle_2mm -> Custom_Electrode:A2_B2
- U23: footprint Custom_Electrode:Circle_2mm -> Custom_Electrode:A2_C3
- U24: footprint Custom_Electrode:Circle_2mm -> Custom_Electrode:A2_C#3
- U25: footprint Custom_Electrode:Circle_2mm -> Custom_Electrode:A2_D3
- U26: footprint Custom_Electrode:Circle_2mm -> Custom_Electrode:A2_D#3
- U27: footprint Custom_Electrode:Circle_2mm -> Custom_Electrode:A2_E3
- U28: footprint Custom_Electrode:Circle_2mm -> Custom_Electrode:A2_F3
- U29: footprint Custom_Electrode:Circle_2mm -> Custom_Electrode:A2_F#3
- U30: footprint Custom_Electrode:Circle_2mm -> Custom_Electrode:A2_G3
- U31: footprint Custom_Electrode:Circle_2mm -> Custom_Electrode:A2_G#3
- U32: footprint Custom_Electrode:Circle_2mm -> Custom_Electrode:A2_A3
- U33: footprint Custom_Electrode:Circle_2mm -> Custom_Electrode:A2_A#3
- U34: footprint Custom_Electrode:Circle_2mm -> Custom_Electrode:A2_B3
- U35: footprint Custom_Electrode:Circle_2mm -> Custom_Electrode:A2_C4
- U36: footprint Custom_Electrode:Circle_2mm -> Custom_Electrode:A2_C#4
- U37: footprint Custom_Electrode:Circle_2mm -> Custom_Electrode:A2_D4
- U38: footprint Custom_Electrode:Circle_2mm -> Custom_Electrode:A2_D#4
- U39: footprint Custom_Electrode:Circle_2mm -> Custom_Electrode:A2_E4
- U40: footprint Custom_Electrode:Circle_2mm -> Custom_Electrode:A2_F4
- U41: footprint Custom_Electrode:Circle_2mm -> Custom_Electrode:D3_D#3
- U42: footprint Custom_Electrode:Circle_2mm -> Custom_Electrode:D3_E3
- U43: footprint Custom_Electrode:Circle_2mm -> Custom_Electrode:D3_F3
- U44: footprint Custom_Electrode:Circle_2mm -> Custom_Electrode:D3_F#3
- U45: footprint Custom_Electrode:Circle_2mm -> Custom_Electrode:D3_G3
- U46: footprint Custom_Electrode:Circle_2mm -> Custom_Electrode:D3_G#3
- U47: footprint Custom_Electrode:Circle_2mm -> Custom_Electrode:D3_A3
- U48: footprint Custom_Electrode:Circle_2mm -> Custom_Electrode:D3_A#3
- U49: footprint Custom_Electrode:Circle_2mm -> Custom_Electrode:D3_B3
- U50: footprint Custom_Electrode:Circle_2mm -> Custom_Electrode:D3_C4
- U51: footprint Custom_Electrode:Circle_2mm -> Custom_Electrode:D3_C#4
- U52: footprint Custom_Electrode:Circle_2mm -> Custom_Electrode:D3_D4
- U53: footprint Custom_Electrode:Circle_2mm -> Custom_Electrode:D3_D#4
- U54: footprint Custom_Electrode:Circle_2mm -> Custom_Electrode:D3_E4
- U55: footprint Custom_Electrode:Circle_2mm -> Custom_Electrode:D3_F4
- U56: footprint Custom_Electrode:Circle_2mm -> Custom_Electrode:D3_F#4
- U57: footprint Custom_Electrode:Circle_2mm -> Custom_Electrode:D3_G4
- U58: footprint Custom_Electrode:Circle_2mm -> Custom_Electrode:D3_G#4
- U59: footprint Custom_Electrode:Circle_2mm -> Custom_Electrode:D3_A4
- U60: footprint Custom_Electrode:Circle_2mm -> Custom_Electrode:D3_A#4
- U61: footprint Custom_Electrode:Circle_2mm -> Custom_Electrode:G3_G#3
- U62: footprint Custom_Electrode:Circle_2mm -> Custom_Electrode:G3_A3
- U63: footprint Custom_Electrode:Circle_2mm -> Custom_Electrode:G3_A#3
- U64: footprint Custom_Electrode:Circle_2mm -> Custom_Electrode:G3_B3
- U65: footprint Custom_Electrode:Circle_2mm -> Custom_Electrode:G3_C4
- U66: footprint Custom_Electrode:Circle_2mm -> Custom_Electrode:G3_C#4
- U67: footprint Custom_Electrode:Circle_2mm -> Custom_Electrode:G3_D4
- U68: footprint Custom_Electrode:Circle_2mm -> Custom_Electrode:G3_D#4
- U69: footprint Custom_Electrode:Circle_2mm -> Custom_Electrode:G3_E4
- U70: footprint Custom_Electrode:Circle_2mm -> Custom_Electrode:G3_F4
- U71: footprint Custom_Electrode:Circle_2mm -> Custom_Electrode:G3_F#4
- U72: footprint Custom_Electrode:Circle_2mm -> Custom_Electrode:G3_G4
- U73: footprint Custom_Electrode:Circle_2mm -> Custom_Electrode:G3_G#4
- U74: footprint Custom_Electrode:Circle_2mm -> Custom_Electrode:G3_A4
- U75: footprint Custom_Electrode:Circle_2mm -> Custom_Electrode:G3_A#4
- U76: footprint Custom_Electrode:Circle_2mm -> Custom_Electrode:G3_B4
- U77: footprint Custom_Electrode:Circle_2mm -> Custom_Electrode:G3_C5
- U78: footprint Custom_Electrode:Circle_2mm -> Custom_Electrode:G3_C#5
- U79: footprint Custom_Electrode:Circle_2mm -> Custom_Electrode:G3_D5
- U80: footprint Custom_Electrode:Circle_2mm -> Custom_Electrode:G3_D#5
- moved U61 526.6 mm to (24.0, 1.20)
- moved U41 521.6 mm to (16.1, 1.15)
- moved U21 512.8 mm to (8.35, 1.15)
- moved U62 492.8 mm to (24.1, 38.0)
- moved U42 492.2 mm to (16.1, 38.0)
- moved U22 482.8 mm to (8.20, 38.0)
- moved U63 465.5 mm to (24.1, 72.5)
- moved U43 464.0 mm to (16.1, 72.5)
- moved U44 455.7 mm to (16.1, 104.9)
- moved U23 455.4 mm to (7.90, 72.5)
- moved U64 437.4 mm to (24.3, 104.9)
- moved U45 433.1 mm to (15.9, 135.6)
- moved U24 430.6 mm to (7.65, 104.9)
- moved U65 414.9 mm to (24.4, 135.6)
- moved U46 413.0 mm to (16.0, 164.5)
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
Commit message: Added all frets on pcb
Parts:
- U100: footprint Custom_Electrode:Circle_2mm -> Custom_Electrode:B3_G5
- U101: footprint Custom_Electrode:Circle_2mm -> Custom_Electrode:E4_F4
- U102: footprint Custom_Electrode:Circle_2mm -> Custom_Electrode:E4_F#4
- U103: footprint Custom_Electrode:Circle_2mm -> Custom_Electrode:E4_G4
- U104: footprint Custom_Electrode:Circle_2mm -> Custom_Electrode:E4_G#4
- U105: footprint Custom_Electrode:Circle_2mm -> Custom_Electrode:E4_A4
- U106: footprint Custom_Electrode:Circle_2mm -> Custom_Electrode:E4_A#4
- U107: footprint Custom_Electrode:Circle_2mm -> Custom_Electrode:E4_B4
- U108: footprint Custom_Electrode:Circle_2mm -> Custom_Electrode:E4_C5
- U109: footprint Custom_Electrode:Circle_2mm -> Custom_Electrode:E4_C#5
- U110: footprint Custom_Electrode:Circle_2mm -> Custom_Electrode:E4_D5
- U111: footprint Custom_Electrode:Circle_2mm -> Custom_Electrode:E4_D#5
- U112: footprint Custom_Electrode:Circle_2mm -> Custom_Electrode:E4_E5
- U113: footprint Custom_Electrode:Circle_2mm -> Custom_Electrode:E4_F5
- U114: footprint Custom_Electrode:Circle_2mm -> Custom_Electrode:E4_F#5
- U115: footprint Custom_Electrode:Circle_2mm -> Custom_Electrode:E4_G5
- U116: footprint Custom_Electrode:Circle_2mm -> Custom_Electrode:E4_G#5
- U117: footprint Custom_Electrode:Circle_2mm -> Custom_Electrode:E4_A5
- U118: footprint Custom_Electrode:Circle_2mm -> Custom_Electrode:E4_A#5
- U119: footprint Custom_Electrode:Circle_2mm -> Custom_Electrode:E4_B5
- U120: footprint Custom_Electrode:E4_Fret20 -> Custom_Electrode:E4_C6
- U81: footprint Custom_Electrode:Circle_2mm -> Custom_Electrode:B3_C4
- U82: footprint Custom_Electrode:Circle_2mm -> Custom_Electrode:B3_C#4
- U83: footprint Custom_Electrode:Circle_2mm -> Custom_Electrode:B3_D4
- U84: footprint Custom_Electrode:Circle_2mm -> Custom_Electrode:B3_D#4
- U85: footprint Custom_Electrode:Circle_2mm -> Custom_Electrode:B3_E4
- U86: footprint Custom_Electrode:Circle_2mm -> Custom_Electrode:B3_F4
- U87: footprint Custom_Electrode:Circle_2mm -> Custom_Electrode:B3_F#4
- U88: footprint Custom_Electrode:Circle_2mm -> Custom_Electrode:B3_G4
- U89: footprint Custom_Electrode:Circle_2mm -> Custom_Electrode:B3_G#4
- U90: footprint Custom_Electrode:Circle_2mm -> Custom_Electrode:B3_A4
- U91: footprint Custom_Electrode:Circle_2mm -> Custom_Electrode:B3_A#4
- U92: footprint Custom_Electrode:Circle_2mm -> Custom_Electrode:B3_B4
- U93: footprint Custom_Electrode:Circle_2mm -> Custom_Electrode:B3_C5
- U94: footprint Custom_Electrode:Circle_2mm -> Custom_Electrode:B3_C#5
- U95: footprint Custom_Electrode:Circle_2mm -> Custom_Electrode:B3_D5
- U96: footprint Custom_Electrode:Circle_2mm -> Custom_Electrode:B3_D#5
- U97: footprint Custom_Electrode:Circle_2mm -> Custom_Electrode:B3_E5
- U98: footprint Custom_Electrode:Circle_2mm -> Custom_Electrode:B3_F5
- U99: footprint Custom_Electrode:Circle_2mm -> Custom_Electrode:B3_F#5
- moved U100 355.4 mm to (34.5, 434.6)
- moved U119 354.0 mm to (44.1, 421.7)
- moved U118 349.6 mm to (44.0, 408.1)
- moved U99 348.8 mm to (34.8, 421.7)
- moved U117 339.4 mm to (43.9, 393.8)
- moved U98 336.2 mm to (34.6, 408.1)
- moved U96 333.9 mm to (34.5, 378.2)
- moved U97 328.9 mm to (34.6, 393.8)
- moved U116 328.6 mm to (43.6, 378.2)
- moved U101 324.7 mm to (38.9, 1.20)
- moved U95 319.9 mm to (34.2, 361.9)
- moved U115 314.9 mm to (43.5, 361.9)
- moved U83 310.5 mm to (32.2, 72.8)
- moved U102 302.6 mm to (39.3, 38.0)
- moved U112 300.3 mm to (42.8, 307.4)
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
Commit message: Tracing is31se5100
Parts:
- removed J1, J2, J3, J4, J5, J6: Conn_01x20, Connector_PinHeader_2.54mm:PinHeader_1x20_P2.54mm_Vertical
- added U1: IS31SE5100-SALS2, Package_SO:SSOP-24_5.3x8.2mm_P0.65mm, B.Cu at (11.0, 142.7)
- added U121: IS31SE5100-SALS2, Package_SO:SSOP-24_5.3x8.2mm_P0.65mm, B.Cu at (8.30, 127.8)
- added U122: IS31SE5100-SALS2, Package_SO:SSOP-24_5.3x8.2mm_P0.65mm, B.Cu at (7.25, 274.1)
- added U123: IS31SE5100-SALS2, Package_SO:SSOP-24_5.3x8.2mm_P0.65mm, B.Cu at (3.40, 418.9)
- added U125: IS31SE5100-SALS2, Package_SO:SSOP-24_5.3x8.2mm_P0.65mm, B.Cu at (6.35, 287.2)
- added U126: IS31SE5100-SALS2, Package_SO:SSOP-24_5.3x8.2mm_P0.65mm, B.Cu at (3.65, 431.6)
- added U127: IS31SE5100-SALS2, Package_SO:SSOP-24_5.3x8.2mm_P0.65mm, B.Cu at (15.0, 157.0)
- added U128: IS31SE5100-SALS2, Package_SO:SSOP-24_5.3x8.2mm_P0.65mm, B.Cu at (-128.3, 107.5)
- added U129: IS31SE5100-SALS2, Package_SO:SSOP-24_5.3x8.2mm_P0.65mm, B.Cu at (-117.8, 97.5)
- added U130: IS31SE5100-SALS2, Package_SO:SSOP-24_5.3x8.2mm_P0.65mm, B.Cu at (27.1, 112.0)
- added U131: IS31SE5100-SALS2, Package_SO:SSOP-24_5.3x8.2mm_P0.65mm, B.Cu at (-138.8, 87.4)
- added U132: IS31SE5100-SALS2, Package_SO:SSOP-24_5.3x8.2mm_P0.65mm, B.Cu at (-107.2, 97.5)
- added U133: IS31SE5100-SALS2, Package_SO:SSOP-24_5.3x8.2mm_P0.65mm, B.Cu at (30.6, 157.2)
- added U134: IS31SE5100-SALS2, Package_SO:SSOP-24_5.3x8.2mm_P0.65mm, B.Cu at (-107.2, 107.5)
- added U135: IS31SE5100-SALS2, Package_SO:SSOP-24_5.3x8.2mm_P0.65mm, B.Cu at (-96.7, 97.5)
- added U136: IS31SE5100-SALS2, Package_SO:SSOP-24_5.3x8.2mm_P0.65mm, B.Cu at (40.0, 130.8)
- added U137: IS31SE5100-SALS2, Package_SO:SSOP-24_5.3x8.2mm_P0.65mm, B.Cu at (-96.7, 107.5)
- added U138: IS31SE5100-SALS2, Package_SO:SSOP-24_5.3x8.2mm_P0.65mm, B.Cu at (-86.1, 97.5)
- added U139: MAX7301, Custom:MAX7301AAX, B.Cu at (10.3, 235.6)
Connections:
- U1 pad 1: Net-(J1-Pad1) -> /Electrode_1
- U10 pad 1: Net-(J1-Pad10) -> /Electrode_10
- U100 pad 1: Net-(J5-Pad20) -> /Electrode_100
- U101 pad 1: Net-(J6-Pad1) -> /Electrode_101
- U102 pad 1: Net-(J6-Pad2) -> /Electrode_102
- U103 pad 1: Net-(J6-Pad3) -> /Electrode_103
- U104 pad 1: Net-(J6-Pad4) -> /Electrode_104
- U105 pad 1: Net-(J6-Pad5) -> /Electrode_105
- U106 pad 1: Net-(J6-Pad6) -> /Electrode_106
- U107 pad 1: Net-(J6-Pad7) -> /Electrode_107
- U108 pad 1: Net-(J6-Pad8) -> /Electrode_108
- U109 pad 1: Net-(J6-Pad9) -> /Electrode_109
- U11 pad 1: Net-(J1-Pad11) -> /Electrode_11
- U110 pad 1: Net-(J6-Pad10) -> /Electrode_110
- U111 pad 1: Net-(J6-Pad11) -> /Electrode_111
- U112 pad 1: Net-(J6-Pad12) -> /Electrode_112
- U113 pad 1: Net-(J6-Pad13) -> /Electrode_113
- U114 pad 1: Net-(J6-Pad14) -> /Electrode_114
- U115 pad 1: Net-(J6-Pad15) -> /Electrode_115
- U116 pad 1: Net-(J6-Pad16) -> /Electrode_116
- U117 pad 1: Net-(J6-Pad17) -> /Electrode_117
- U118 pad 1: Net-(J6-Pad18) -> /Electrode_118
- U119 pad 1: Net-(J6-Pad19) -> /Electrode_119
- U12 pad 1: Net-(J1-Pad12) -> /Electrode_12
- U120 pad 1: Net-(J6-Pad20) -> /Electrode_120
- U13 pad 1: Net-(J1-Pad13) -> /Electrode_13
- U14 pad 1: Net-(J1-Pad14) -> /Electrode_14
- U15 pad 1: Net-(J1-Pad15) -> /Electrode_15
- U16 pad 1: Net-(J1-Pad16) -> /Electrode_16
- U17 pad 1: Net-(J1-Pad17) -> /Electrode_17
- U18 pad 1: Net-(J1-Pad18) -> /Electrode_18
- U19 pad 1: Net-(J1-Pad19) -> /Electrode_19
- U2 pad 1: Net-(J1-Pad2) -> /Electrode_2
- U20 pad 1: Net-(J1-Pad20) -> /Electrode_20
- U21 pad 1: Net-(J2-Pad1) -> /Electrode_21
- U22 pad 1: Net-(J2-Pad2) -> /Electrode_22
- U23 pad 1: Net-(J2-Pad3) -> /Electrode_23
- U24 pad 1: Net-(J2-Pad4) -> /Electrode_24
- U25 pad 1: Net-(J2-Pad5) -> /Electrode_25
- U26 pad 1: Net-(J2-Pad6) -> /Electrode_26
- U27 pad 1: Net-(J2-Pad7) -> /Electrode_27
- U28 pad 1: Net-(J2-Pad8) -> /Electrode_28
- U29 pad 1: Net-(J2-Pad9) -> /Electrode_29
- U3 pad 1: Net-(J1-Pad3) -> /Electrode_3
- U30 pad 1: Net-(J2-Pad10) -> /Electrode_30
- U31 pad 1: Net-(J2-Pad11) -> /Electrode_31
- U32 pad 1: Net-(J2-Pad12) -> /Electrode_32
- U33 pad 1: Net-(J2-Pad13) -> /Electrode_33
- U34 pad 1: Net-(J2-Pad14) -> /Electrode_34
- U35 pad 1: Net-(J2-Pad15) -> /Electrode_35
- U36 pad 1: Net-(J2-Pad16) -> /Electrode_36
- U37 pad 1: Net-(J2-Pad17) -> /Electrode_37
- U38 pad 1: Net-(J2-Pad18) -> /Electrode_38
- U39 pad 1: Net-(J2-Pad19) -> /Electrode_39
- U4 pad 1: Net-(J1-Pad4) -> /Electrode_4
- U40 pad 1: Net-(J2-Pad20) -> /Electrode_40
- U41 pad 1: Net-(J3-Pad1) -> /Electrode_41
- U42 pad 1: Net-(J3-Pad2) -> /Electrode_42
- U43 pad 1: Net-(J3-Pad3) -> /Electrode_43
- U44 pad 1: Net-(J3-Pad4) -> /Electrode_44
- U45 pad 1: Net-(J3-Pad5) -> /Electrode_45
- U46 pad 1: Net-(J3-Pad6) -> /Electrode_46
- U47 pad 1: Net-(J3-Pad7) -> /Electrode_47
- U48 pad 1: Net-(J3-Pad8) -> /Electrode_48
- U49 pad 1: Net-(J3-Pad9) -> /Electrode_49
- U5 pad 1: Net-(J1-Pad5) -> /Electrode_5
- U50 pad 1: Net-(J3-Pad10) -> /Electrode_50
- U51 pad 1: Net-(J3-Pad11) -> /Electrode_51
- U52 pad 1: Net-(J3-Pad12) -> /Electrode_52
- U53 pad 1: Net-(J3-Pad13) -> /Electrode_53
- U54 pad 1: Net-(J3-Pad14) -> /Electrode_54
- U55 pad 1: Net-(J3-Pad15) -> /Electrode_55
- U56 pad 1: Net-(J3-Pad16) -> /Electrode_56
- U57 pad 1: Net-(J3-Pad17) -> /Electrode_57
- U58 pad 1: Net-(J3-Pad18) -> /Electrode_58
- U59 pad 1: Net-(J3-Pad19) -> /Electrode_59
- U6 pad 1: Net-(J1-Pad6) -> /Electrode_6
- U60 pad 1: Net-(J3-Pad20) -> /Electrode_60
- U61 pad 1: Net-(J4-Pad1) -> /Electrode_61
- U62 pad 1: Net-(J4-Pad2) -> /Electrode_62
- U63 pad 1: Net-(J4-Pad3) -> /Electrode_63
- U64 pad 1: Net-(J4-Pad4) -> /Electrode_64
- U65 pad 1: Net-(J4-Pad5) -> /Electrode_65
- U66 pad 1: Net-(J4-Pad6) -> /Electrode_66
- U67 pad 1: Net-(J4-Pad7) -> /Electrode_67
- U68 pad 1: Net-(J4-Pad8) -> /Electrode_68
- U69 pad 1: Net-(J4-Pad9) -> /Electrode_69
- U7 pad 1: Net-(J1-Pad7) -> /Electrode_7
- U70 pad 1: Net-(J4-Pad10) -> /Electrode_70
- U71 pad 1: Net-(J4-Pad11) -> /Electrode_71
- U72 pad 1: Net-(J4-Pad12) -> /Electrode_72
- U73 pad 1: Net-(J4-Pad13) -> /Electrode_73
- U74 pad 1: Net-(J4-Pad14) -> /Electrode_74
- U75 pad 1: Net-(J4-Pad15) -> /Electrode_75
- U76 pad 1: Net-(J4-Pad16) -> /Electrode_76
- U77 pad 1: Net-(J4-Pad17) -> /Electrode_77
- U78 pad 1: Net-(J4-Pad18) -> /Electrode_78
- U79 pad 1: Net-(J4-Pad19) -> /Electrode_79
- U8 pad 1: Net-(J1-Pad8) -> /Electrode_8
- U80 pad 1: Net-(J4-Pad20) -> /Electrode_80
- U81 pad 1: Net-(J5-Pad1) -> /Electrode_81
- U82 pad 1: Net-(J5-Pad2) -> /Electrode_82
- U83 pad 1: Net-(J5-Pad3) -> /Electrode_83
- U84 pad 1: Net-(J5-Pad4) -> /Electrode_84
- U85 pad 1: Net-(J5-Pad5) -> /Electrode_85
- U86 pad 1: Net-(J5-Pad6) -> /Electrode_86
- U87 pad 1: Net-(J5-Pad7) -> /Electrode_87
- U88 pad 1: Net-(J5-Pad8) -> /Electrode_88
- U89 pad 1: Net-(J5-Pad9) -> /Electrode_89
- U9 pad 1: Net-(J1-Pad9) -> /Electrode_9
- U90 pad 1: Net-(J5-Pad10) -> /Electrode_90
- U91 pad 1: Net-(U91-Pad1) -> /Electrode_91
- U92 pad 1: Net-(J5-Pad12) -> /Electrode_92
- U93 pad 1: Net-(J5-Pad13) -> /Electrode_93
- U94 pad 1: Net-(J5-Pad14) -> /Electrode_94
- U95 pad 1: Net-(J5-Pad15) -> /Electrode_95
- U96 pad 1: Net-(J5-Pad16) -> /Electrode_96
- U97 pad 1: Net-(J5-Pad17) -> /Electrode_97
- U98 pad 1: Net-(J5-Pad18) -> /Electrode_98
- U99 pad 1: Net-(J5-Pad19) -> /Electrode_99
Routing:
- net /Electrode_41: track 0.00 -> 183.2 mm, vias 0 -> 1
- net /Electrode_21: track 0.00 -> 171.3 mm, vias 0 -> 1
- net /Electrode_81: track 0.00 -> 152.2 mm, vias 0 -> 1
- net /Electrode_1: track 0.00 -> 151.7 mm, vias 0 -> 1
- net /Electrode_42: track 0.00 -> 150.8 mm, vias 0 -> 1
- net /Electrode_68: track 0.00 -> 138.9 mm, vias 0 -> 1
- net /Electrode_22: track 0.00 -> 134.4 mm, vias 0 -> 1
- net /Electrode_61: track 0.00 -> 129.0 mm, vias 0 -> 1
- net /Electrode_82: track 0.00 -> 127.1 mm, vias 0 -> 1
- net /Electrode_43: track 0.00 -> 117.5 mm, vias 0 -> 1
- net /Electrode_2: track 0.00 -> 114.9 mm, vias 0 -> 1
- net /Electrode_8: track 0.00 -> 111.9 mm, vias 0 -> 1
- net /Electrode_83: track 0.00 -> 108.7 mm, vias 0 -> 1
- net /Electrode_23: track 0.00 -> 101.5 mm, vias 0 -> 1
- net /Electrode_67: track 0.00 -> 97.6 mm, vias 0 -> 1
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Other:
- copper layers 2 -> 4
