File: capacitive_fingerboard_guitar_650/capacitive_fingerboard_guitar_650.kicad_pcb (KiCad board)
At the start: 4 copper layers, 60.6 x 500 mm, 139 parts, among them U1 Electrode, U1 IS31SE5100-SALS2, U10 Electrode, U100 Electrode, U101 Electrode, U102 Electrode, U103 Electrode, U104 Electrode, U105 Electrode, U106 Electrode, U107 Electrode, U108 Electrode, U109 Electrode, U11 Electrode, U110 Electrode, U111 Electrode, U112 Electrode, U113 Electrode, U114 Electrode, U115 Electrode, U116 Electrode, U117 Electrode, U118 Electrode, U119 Electrode, U12 Electrode, U120 Electrode, U121 IS31SE5100-SALS2, U122 IS31SE5100-SALS2, U123 IS31SE5100-SALS2, U125 IS31SE5100-SALS2, U126 IS31SE5100-SALS2, U127 IS31SE5100-SALS2, U128 IS31SE5100-SALS2, U129 IS31SE5100-SALS2, U13 Electrode, U130 IS31SE5100-SALS2, U131 IS31SE5100-SALS2, U132 IS31SE5100-SALS2, U133 IS31SE5100-SALS2, U134 IS31SE5100-SALS2, U135 IS31SE5100-SALS2, U136 IS31SE5100-SALS2, U137 IS31SE5100-SALS2, U138 IS31SE5100-SALS2, U139 MAX7301, U14 Electrode, U15 Electrode, U16 Electrode, U17 Electrode, U18 Electrode, U19 Electrode, U2 Electrode, U20 Electrode, U21 Electrode, U22 Electrode, U23 Electrode, U24 Electrode, U25 Electrode, U26 Electrode, U27 Electrode, U28 Electrode, U29 Electrode, U3 Electrode, U30 Electrode, U31 Electrode, U32 Electrode, U33 Electrode, U34 Electrode, U35 Electrode, U36 Electrode, U37 Electrode, U38 Electrode, U39 Electrode, U4 Electrode, U40 Electrode, U41 Electrode, U42 Electrode, U43 Electrode, U44 Electrode, U45 Electrode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

Commit message: Added traces for the first third
Parts:
- removed the U1 at (11.0, 142.7)
- removed U121, U122, U123, U125, U126, U127, U128, U129, U130, U131, U132, U133, U134, U135, U136, U137, U138: IS31SE5100-SALS2, Package_SO:SSOP-24_5.3x8.2mm_P0.65mm
- removed U139: MAX7301, Custom:MAX7301AAX
- added J1: Conn_01x08, Custom:SAMTEC_TSM-108-01-F-SV, B.Cu at (3.91, 132.8)
- added J10: Conn_01x08, Custom:SAMTEC_TSM-108-01-F-SV, B.Cu at (22.9, 149.2)
- added J11: Conn_02x04_Top_Bottom, Connector_Harwin:Harwin_M20-7810445_2x04_P2.54mm_Vertical, B.Cu at (-94.8, 114.3)
- added J12: Conn_02x04_Top_Bottom, Connector_Harwin:Harwin_M20-7810445_2x04_P2.54mm_Vertical, B.Cu at (-104.5, 126.6)
- added J13: Conn_01x08, Custom:SAMTEC_TSM-108-01-F-SV, B.Cu at (30.5, 119.4)
- added J14: Conn_02x04_Top_Bottom, Connector_Harwin:Harwin_M20-7810445_2x04_P2.54mm_Vertical, B.Cu at (-104.5, 138.8)
- added J15: Conn_02x04_Top_Bottom, Connector_Harwin:Harwin_M20-7810445_2x04_P2.54mm_Vertical, B.Cu at (-85.2, 114.3)
- added J16: Conn_01x08, Custom:SAMTEC_TSM-108-01-F-SV, B.Cu at (39.6, 150.0)
- added J17: Conn_02x04_Top_Bottom, Connector_Harwin:Harwin_M20-7810445_2x04_P2.54mm_Vertical, B.Cu at (-75.5, 114.3)
- added J18: Conn_02x04_Top_Bottom, Connector_Harwin:Harwin_M20-7810445_2x04_P2.54mm_Vertical, B.Cu at (-85.2, 126.6)
- added J2: Conn_02x04_Top_Bottom, Connector_Harwin:Harwin_M20-7810445_2x04_P2.54mm_Vertical, B.Cu at (-41.3, 147.0)
- added J3: Conn_02x04_Top_Bottom, Connector_Harwin:Harwin_M20-7810445_2x04_P2.54mm_Vertical, B.Cu at (-41.9, 130.3)
- added J4: Conn_01x08, Custom:SAMTEC_TSM-108-01-F-SV, B.Cu at (13.7, 122.0)
- added J5: Conn_02x04_Top_Bottom, Connector_Harwin:Harwin_M20-7810445_2x04_P2.54mm_Vertical, B.Cu at (-114.1, 114.3)
- added J6: Conn_02x04_Top_Bottom, Connector_Harwin:Harwin_M20-7810445_2x04_P2.54mm_Vertical, B.Cu at (-123.8, 126.6)
- added J7: Conn_01x08, Custom:SAMTEC_TSM-108-01-F-SV, B.Cu at (16.0, 100.0)
- added J8: Conn_02x04_Top_Bottom, Connector_Harwin:Harwin_M20-7810445_2x04_P2.54mm_Vertical, B.Cu at (-123.8, 138.8)
- added J9: Conn_02x04_Top_Bottom, Connector_Harwin:Harwin_M20-7810445_2x04_P2.54mm_Vertical, B.Cu at (-104.5, 114.3)
Routing:
- net /Electrode_101: track 0.00 -> 142.9 mm, vias 0 -> 1
- net /Electrode_48: track 13.3 -> 145.5 mm
- net /Electrode_102: track 0.00 -> 100.9 mm, vias 0 -> 1
- net /Electrode_42: track 150.8 -> 50.9 mm
- net /Electrode_41: track 183.2 -> 93.5 mm
- net /Electrode_108: track 0.00 -> 84.5 mm, vias 0 -> 1
- net /Electrode_43: track 117.5 -> 45.9 mm
- net /Electrode_83: track 108.7 -> 37.3 mm
- net /Electrode_23: track 101.5 -> 34.7 mm
- net /Electrode_22: track 134.4 -> 70.0 mm
- net /Electrode_46: track 20.5 -> 84.1 mm
- net /Electrode_103: track 0.00 -> 60.1 mm, vias 0 -> 1
- net /Electrode_21: track 171.3 -> 113.0 mm
- net /Electrode_88: track 64.0 -> 122.3 mm
- net /Electrode_107: track 0.00 -> 58.1 mm, vias 0 -> 1
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
Commit message: Added missing trace
Parts:
- moved J13 1.50 mm to (32.0, 119.4)
Routing:
- net /Electrode_47: track 0.00 -> 117.3 mm, vias 0 -> 1
- net /Electrode_83: track 37.3 -> 27.9 mm
- net /Electrode_63: track 69.2 -> 59.8 mm
- net /Electrode_81: track 113.1 -> 105.4 mm
- net /Electrode_87: track 94.1 -> 87.3 mm
- net /Electrode_86: track 58.9 -> 52.9 mm
- net /Electrode_85: track 24.9 -> 20.7 mm
- net /Electrode_62: track 102.8 -> 98.7 mm
- net /Electrode_82: track 71.4 -> 68.4 mm
- net /Electrode_61: track 139.1 -> 136.4 mm
- net /Electrode_88: track 122.3 -> 119.6 mm
- net /Electrode_45: track 45.1 -> 47.8 mm
- net /Electrode_23: track 34.7 -> 37.2 mm
- net /Electrode_46: track 84.1 -> 86.1 mm
- net /Electrode_48: track 145.5 -> 147.4 mm
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
Commit message: Over 50% trace done
Parts:
- J11, J12, J14, J15, J17, J18, J2, J3, J5, J6, J8, J9: value Conn_02x04_Top_Bottom -> Conn_01x08; footprint Connector_Harwin:Harwin_M20-7810445_2x04_P2.54mm_Vertical -> Custom:SAMTEC_TSM-108-01-F-SV
- moved J15 374.1 mm to (38.4, 467.4), turned to 90 degrees
- moved J11 373.9 mm to (27.6, 467.6), turned to 90 degrees
- moved J17 373.7 mm to (48.0, 467.0), turned to 270 degrees
- moved J5 372.3 mm to (0.90, 468.4), turned to 270 degrees
- moved J8 356.1 mm to (11.2, 468.3), turned to 270 degrees
- moved J3 338.0 mm to (-12.1, 466.9), turned to 270 degrees
- moved J14 264.8 mm to (80.8, 328.0), turned to 90 degrees
- moved J9 259.5 mm to (14.8, 344.9), turned to 90 degrees
- moved J18 252.2 mm to (41.6, 344.6), turned to 90 degrees
- moved J6 235.8 mm to (12.5, 319.0), turned to 90 degrees
- moved J12 233.9 mm to (26.9, 320.1), turned to 90 degrees
- moved J2 183.0 mm to (1.00, 325.0)
Connections:
- J11 pad 1: /Electrode_69 -> /Electrode_80
- J11 pad 2: /Electrode_70 -> /Electrode_79
- J11 pad 3: /Electrode_71 -> /Electrode_78
- J11 pad 4: /Electrode_72 -> /Electrode_77
- J11 pad 5: /Electrode_73 -> Net-(J11-Pad5)
- J11 pad 6: /Electrode_74 -> Net-(J11-Pad6)
- J11 pad 7: /Electrode_75 -> Net-(J11-Pad7)
- J11 pad 8: /Electrode_76 -> Net-(J11-Pad8)
- J12 pad 1: /Electrode_77 -> /Electrode_72
- J12 pad 2: /Electrode_78 -> /Electrode_71
- J12 pad 3: /Electrode_79 -> /Electrode_70
- J12 pad 4: /Electrode_80 -> /Electrode_69
- J12 pad 5: Net-(J12-Pad5) -> /Electrode_76
- J12 pad 6: Net-(J12-Pad6) -> /Electrode_75
- J12 pad 7: Net-(J12-Pad7) -> /Electrode_74
- J12 pad 8: Net-(J12-Pad8) -> /Electrode_73
- J14 pad 1: /Electrode_89 -> /Electrode_92
- J14 pad 2: /Electrode_90 -> /Electrode_91
- J14 pad 3: /Electrode_91 -> /Electrode_90
- J14 pad 4: /Electrode_92 -> /Electrode_89
- J14 pad 5: /Electrode_93 -> /Electrode_96
- J14 pad 6: /Electrode_94 -> /Electrode_95
- J14 pad 7: /Electrode_95 -> /Electrode_94
- J14 pad 8: /Electrode_96 -> /Electrode_93
- J15 pad 1: /Electrode_97 -> /Electrode_100
- J15 pad 2: /Electrode_98 -> /Electrode_99
- J15 pad 3: /Electrode_99 -> /Electrode_98
- J15 pad 4: /Electrode_100 -> /Electrode_97
- J17 pad 1: /Electrode_109 -> /Electrode_120
- J17 pad 2: /Electrode_110 -> /Electrode_119
- J17 pad 3: /Electrode_111 -> /Electrode_118
- J17 pad 4: /Electrode_112 -> /Electrode_117
- J17 pad 5: /Electrode_113 -> Net-(J17-Pad5)
- J17 pad 6: /Electrode_114 -> Net-(J17-Pad6)
- J17 pad 7: /Electrode_115 -> Net-(J17-Pad7)
- J17 pad 8: /Electrode_116 -> Net-(J17-Pad8)
- J18 pad 1: /Electrode_117 -> /Electrode_112
- J18 pad 2: /Electrode_118 -> /Electrode_111
- J18 pad 3: /Electrode_119 -> /Electrode_110
- J18 pad 4: /Electrode_120 -> /Electrode_109
- J18 pad 5: Net-(J18-Pad5) -> /Electrode_116
- J18 pad 6: Net-(J18-Pad6) -> /Electrode_115
- J18 pad 7: Net-(J18-Pad7) -> /Electrode_114
- J18 pad 8: Net-(J18-Pad8) -> /Electrode_113
- J2 pad 1: /Electrode_9 -> /Electrode_12
- J2 pad 2: /Electrode_10 -> /Electrode_11
- J2 pad 3: /Electrode_11 -> /Electrode_10
- J2 pad 4: /Electrode_12 -> /Electrode_9
- J2 pad 5: /Electrode_13 -> /Electrode_16
- J2 pad 6: /Electrode_14 -> /Electrode_15
- J2 pad 7: /Electrode_15 -> /Electrode_14
- J2 pad 8: /Electrode_16 -> /Electrode_13
- J3 pad 1: /Electrode_17 -> /Electrode_20
- J3 pad 2: /Electrode_18 -> /Electrode_19
- J3 pad 3: /Electrode_19 -> /Electrode_18
- J3 pad 4: /Electrode_20 -> /Electrode_17
- J5 pad 1: /Electrode_29 -> /Electrode_40
- J5 pad 2: /Electrode_30 -> /Electrode_39
- J5 pad 3: /Electrode_31 -> /Electrode_38
- J5 pad 4: /Electrode_32 -> /Electrode_37
- J5 pad 5: /Electrode_33 -> Net-(J5-Pad5)
- J5 pad 6: /Electrode_34 -> Net-(J5-Pad6)
- J5 pad 7: /Electrode_35 -> Net-(J5-Pad7)
- J5 pad 8: /Electrode_36 -> Net-(J5-Pad8)
- J6 pad 1: /Electrode_37 -> /Electrode_32
- J6 pad 2: /Electrode_38 -> /Electrode_31
- J6 pad 3: /Electrode_39 -> /Electrode_30
- J6 pad 4: /Electrode_40 -> /Electrode_29
- J6 pad 5: Net-(J6-Pad5) -> /Electrode_36
- J6 pad 6: Net-(J6-Pad6) -> /Electrode_35
- J6 pad 7: Net-(J6-Pad7) -> /Electrode_34
- J6 pad 8: Net-(J6-Pad8) -> /Electrode_33
- J8 pad 1: /Electrode_49 -> /Electrode_60
- J8 pad 2: /Electrode_50 -> /Electrode_59
- J8 pad 3: /Electrode_51 -> /Electrode_58
- J8 pad 4: /Electrode_52 -> /Electrode_57
- J8 pad 5: /Electrode_53 -> Net-(J8-Pad5)
- J8 pad 6: /Electrode_54 -> Net-(J8-Pad6)
- J8 pad 7: /Electrode_55 -> Net-(J8-Pad7)
- J8 pad 8: /Electrode_56 -> Net-(J8-Pad8)
- J9 pad 1: /Electrode_57 -> /Electrode_52
- J9 pad 2: /Electrode_58 -> /Electrode_51
- J9 pad 3: /Electrode_59 -> /Electrode_50
- J9 pad 4: /Electrode_60 -> /Electrode_49
- J9 pad 5: Net-(J9-Pad5) -> /Electrode_56
- J9 pad 6: Net-(J9-Pad6) -> /Electrode_55
- J9 pad 7: Net-(J9-Pad7) -> /Electrode_54
- J9 pad 8: Net-(J9-Pad8) -> /Electrode_53
Routing:
- net /Electrode_49: track 0.00 -> 97.4 mm, vias 0 -> 1
- net /Electrode_9: track 0.00 -> 79.7 mm, vias 0 -> 1
- net /Electrode_36: track 0.00 -> 76.7 mm, vias 0 -> 1
- net /Electrode_50: track 0.00 -> 74.0 mm, vias 0 -> 1
- net /Electrode_29: track 0.00 -> 72.8 mm, vias 0 -> 1
- net /Electrode_16: track 0.00 -> 66.5 mm, vias 0 -> 1
- net /Electrode_10: track 0.00 -> 56.1 mm, vias 0 -> 1
- net /Electrode_35: track 0.00 -> 54.7 mm, vias 0 -> 1
- net /Electrode_15: track 0.00 -> 46.8 mm, vias 0 -> 1
- net /Electrode_51: track 0.00 -> 46.2 mm, vias 0 -> 1
- net /Electrode_70: track 0.00 -> 46.0 mm, vias 0 -> 1
- net /Electrode_30: track 0.00 -> 45.9 mm, vias 0 -> 1
- net /Electrode_56: track 0.00 -> 45.4 mm, vias 0 -> 1
- net /Electrode_52: track 0.00 -> 43.9 mm, vias 0 -> 1
- net /Electrode_34: track 0.00 -> 31.1 mm, vias 0 -> 1
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