File: capacitive_fingerboard_guitar_650/capacitive_fingerboard_guitar_650.sch (KiCad schematic (older format))
At the start: 24 parts, among them J1 Conn_01x20, J2 Conn_01x20, J3 Conn_01x20, J4 Conn_01x20, U1 Electrode, U10 Electrode, U11 Electrode, U12 Electrode, U13 Electrode, U14 Electrode, U15 Electrode, U16 Electrode, U17 Electrode, U18 Electrode, U19 Electrode, U2 Electrode, U20 Electrode, U3 Electrode, U4 Electrode, U5 Electrode, U6 Electrode, U7 Electrode, U8 Electrode, U9 Electrode

Commit message: Added frets on E2 string
Parts:
- added J5, J6: Conn_01x20, Connector_PinHeader_2.54mm:PinHeader_1x20_P2.54mm_Vertical, symbol Connector_Generic:Conn_01x20
- added U100, U101, U102, U103, U104, U105, U106, U107, U108, U109, U110, U111, U112, U113, U114, U115, U116, U117, U118, U119, U21, U22, U23, U24, U25, U26, U27, U28, U29, U30, U31, U32, U33, U34, U35, U36, U37, U38, U39, U40, U41, U42, U43, U44, U45, U46, U47, U48, U49, U50, U51, U52, U53, U54, U55, U56, U57, U58, U59, U60, U61, U62, U63, U64, U65, U66, U67, U68, U69, U70, U71, U72, U73, U74, U75, U76, U77, U78, U79, U80, U81, U82, U83, U84, U85, U86, U87, U88, U89, U90, U91, U92, U93, U94, U95, U96, U97, U98, U99: Electrode, Custom_Electrode:Circle_2mm, symbol Custom_Sensor_Touch:Electrode
- added U120: Electrode, Custom_Electrode:E4_Fret20, symbol Custom_Sensor_Touch:Electrode
- U1: footprint Custom_Electrode:String_1.1684x36.482mm -> Custom_Electrode:E2_F2
- U10: footprint Custom_Electrode:Circle_2mm -> Custom_Electrode:E2_D3
- U11: footprint Custom_Electrode:Circle_2mm -> Custom_Electrode:E2_D#3
- U12: footprint Custom_Electrode:Circle_2mm -> Custom_Electrode:E2_E3
- U13: footprint Custom_Electrode:Circle_2mm -> Custom_Electrode:E2_F3
- U14: footprint Custom_Electrode:Circle_2mm -> Custom_Electrode:E2_F#3
- U15: footprint Custom_Electrode:Circle_2mm -> Custom_Electrode:E2_G3
- U16: footprint Custom_Electrode:Circle_2mm -> Custom_Electrode:E2_G#3
- U17: footprint Custom_Electrode:Circle_2mm -> Custom_Electrode:E2_A3
- U18: footprint Custom_Electrode:Circle_2mm -> Custom_Electrode:E2_A#3
- U19: footprint Custom_Electrode:Circle_2mm -> Custom_Electrode:E2_B3
- U2: footprint Custom_Electrode:Circle_2mm -> Custom_Electrode:E2_F#2
- U20: footprint Custom_Electrode:Circle_2mm -> Custom_Electrode:E2_C4
- U3: footprint Custom_Electrode:Circle_2mm -> Custom_Electrode:E2_G2
- U4: footprint Custom_Electrode:Circle_2mm -> Custom_Electrode:E2_G#2
- U5: footprint Custom_Electrode:Circle_2mm -> Custom_Electrode:E2_A2
- U6: footprint Custom_Electrode:Circle_2mm -> Custom_Electrode:E2_A#2
- U7: footprint Custom_Electrode:Circle_2mm -> Custom_Electrode:E2_B2
- U8: footprint Custom_Electrode:Circle_2mm -> Custom_Electrode:E2_C3
- U9: footprint Custom_Electrode:Circle_2mm -> Custom_Electrode:E2_C#3
Connections:
- net at J2.1 (Pin_1): now also U21.1
- net at J2.10 (Pin_10): now also U30.1
- net at J2.11 (Pin_11): now also U31.1
- net at J2.12 (Pin_12): now also U32.1
- net at J2.13 (Pin_13): now also U33.1
- net at J2.14 (Pin_14): now also U34.1
- net at J2.15 (Pin_15): now also U35.1
- net at J2.16 (Pin_16): now also U36.1
- net at J2.17 (Pin_17): now also U37.1
- net at J2.18 (Pin_18): now also U38.1
- net at J2.19 (Pin_19): now also U39.1
- net at J2.2 (Pin_2): now also U22.1
- net at J2.20 (Pin_20): now also U40.1
- net at J2.3 (Pin_3): now also U23.1
- net at J2.4 (Pin_4): now also U24.1
- net at J2.5 (Pin_5): now also U25.1
- net at J2.6 (Pin_6): now also U26.1
- net at J2.7 (Pin_7): now also U27.1
- net at J2.8 (Pin_8): now also U28.1
- net at J2.9 (Pin_9): now also U29.1
- net at J3.1 (Pin_1): now also U41.1
- net at J3.10 (Pin_10): now also U50.1
- net at J3.11 (Pin_11): now also U51.1
- net at J3.12 (Pin_12): now also U52.1
- net at J3.13 (Pin_13): now also U53.1
- net at J3.14 (Pin_14): now also U54.1
- net at J3.15 (Pin_15): now also U55.1
- net at J3.16 (Pin_16): now also U56.1
- net at J3.17 (Pin_17): now also U57.1
- net at J3.18 (Pin_18): now also U58.1
- net at J3.19 (Pin_19): now also U59.1
- net at J3.2 (Pin_2): now also U42.1
- net at J3.20 (Pin_20): now also U60.1
- net at J3.3 (Pin_3): now also U43.1
- net at J3.4 (Pin_4): now also U44.1
- net at J3.5 (Pin_5): now also U45.1
- net at J3.6 (Pin_6): now also U46.1
- net at J3.7 (Pin_7): now also U47.1
- net at J3.8 (Pin_8): now also U48.1
- net at J3.9 (Pin_9): now also U49.1
- net at J4.1 (Pin_1): now also U61.1
- net at J4.10 (Pin_10): now also U70.1
- net at J4.11 (Pin_11): now also U71.1
- net at J4.12 (Pin_12): now also U72.1
- net at J4.13 (Pin_13): now also U73.1
- net at J4.14 (Pin_14): now also U74.1
- net at J4.15 (Pin_15): now also U75.1
- net at J4.16 (Pin_16): now also U76.1
- net at J4.17 (Pin_17): now also U77.1
- net at J4.18 (Pin_18): now also U78.1
- net at J4.19 (Pin_19): now also U79.1
- net at J4.2 (Pin_2): now also U62.1
- net at J4.20 (Pin_20): now also U80.1
- net at J4.3 (Pin_3): now also U63.1
- net at J4.4 (Pin_4): now also U64.1
- net at J4.5 (Pin_5): now also U65.1
- net at J4.6 (Pin_6): now also U66.1
- net at J4.7 (Pin_7): now also U67.1
- net at J4.8 (Pin_8): now also U68.1
- net at J4.9 (Pin_9): now also U69.1
- new net: J5.1 (Pin_1), U81.1
- new net: J5.10 (Pin_10), U90.1
- new net: J5.12 (Pin_12), U92.1
- new net: J5.13 (Pin_13), U93.1
- new net: J5.14 (Pin_14), U94.1
- new net: J5.15 (Pin_15), U95.1
- new net: J5.16 (Pin_16), U96.1
- new net: J5.17 (Pin_17), U97.1
- new net: J5.18 (Pin_18), U98.1
- new net: J5.19 (Pin_19), U99.1
- new net: J5.2 (Pin_2), U82.1
- new net: J5.20 (Pin_20), U100.1
- new net: J5.3 (Pin_3), U83.1
- new net: J5.4 (Pin_4), U84.1
- new net: J5.5 (Pin_5), U85.1
- new net: J5.6 (Pin_6), U86.1
- new net: J5.7 (Pin_7), U87.1
- new net: J5.8 (Pin_8), U88.1
- new net: J5.9 (Pin_9), U89.1
- new net: J6.1 (Pin_1), U101.1
- new net: J6.10 (Pin_10), U110.1
- new net: J6.11 (Pin_11), U111.1
- new net: J6.12 (Pin_12), U112.1
- new net: J6.13 (Pin_13), U113.1
- new net: J6.14 (Pin_14), U114.1
- new net: J6.15 (Pin_15), U115.1
- new net: J6.16 (Pin_16), U116.1
- new net: J6.17 (Pin_17), U117.1
- new net: J6.18 (Pin_18), U118.1
- new net: J6.19 (Pin_19), U119.1
- new net: J6.2 (Pin_2), U102.1
- new net: J6.20 (Pin_20), U120.1
- new net: J6.3 (Pin_3), U103.1
- new net: J6.4 (Pin_4), U104.1
- new net: J6.5 (Pin_5), U105.1
- new net: J6.6 (Pin_6), U106.1
- new net: J6.7 (Pin_7), U107.1
- new net: J6.8 (Pin_8), U108.1
- new net: J6.9 (Pin_9), U109.1
- no-connect marks 60 -> 0

Commit message: Added more frets on pcb
Parts:
- U21: footprint Custom_Electrode:Circle_2mm -> Custom_Electrode:A2_A#2
- U22: footprint Custom_Electrode:Circle_2mm -> Custom_Electrode:A2_B2
- U23: footprint Custom_Electrode:Circle_2mm -> Custom_Electrode:A2_C3
- U24: footprint Custom_Electrode:Circle_2mm -> Custom_Electrode:A2_C#3
- U25: footprint Custom_Electrode:Circle_2mm -> Custom_Electrode:A2_D3
- U26: footprint Custom_Electrode:Circle_2mm -> Custom_Electrode:A2_D#3
- U27: footprint Custom_Electrode:Circle_2mm -> Custom_Electrode:A2_E3
- U28: footprint Custom_Electrode:Circle_2mm -> Custom_Electrode:A2_F3
- U29: footprint Custom_Electrode:Circle_2mm -> Custom_Electrode:A2_F#3
- U30: footprint Custom_Electrode:Circle_2mm -> Custom_Electrode:A2_G3
- U31: footprint Custom_Electrode:Circle_2mm -> Custom_Electrode:A2_G#3
- U32: footprint Custom_Electrode:Circle_2mm -> Custom_Electrode:A2_A3
- U33: footprint Custom_Electrode:Circle_2mm -> Custom_Electrode:A2_A#3
- U34: footprint Custom_Electrode:Circle_2mm -> Custom_Electrode:A2_B3
- U35: footprint Custom_Electrode:Circle_2mm -> Custom_Electrode:A2_C4
- U36: footprint Custom_Electrode:Circle_2mm -> Custom_Electrode:A2_C#4
- U37: footprint Custom_Electrode:Circle_2mm -> Custom_Electrode:A2_D4
- U38: footprint Custom_Electrode:Circle_2mm -> Custom_Electrode:A2_D#4
- U39: footprint Custom_Electrode:Circle_2mm -> Custom_Electrode:A2_E4
- U40: footprint Custom_Electrode:Circle_2mm -> Custom_Electrode:A2_F4
- U41: footprint Custom_Electrode:Circle_2mm -> Custom_Electrode:D3_D#3
- U42: footprint Custom_Electrode:Circle_2mm -> Custom_Electrode:D3_E3
- U43: footprint Custom_Electrode:Circle_2mm -> Custom_Electrode:D3_F3
- U44: footprint Custom_Electrode:Circle_2mm -> Custom_Electrode:D3_F#3
- U45: footprint Custom_Electrode:Circle_2mm -> Custom_Electrode:D3_G3
- U46: footprint Custom_Electrode:Circle_2mm -> Custom_Electrode:D3_G#3
- U47: footprint Custom_Electrode:Circle_2mm -> Custom_Electrode:D3_A3
- U48: footprint Custom_Electrode:Circle_2mm -> Custom_Electrode:D3_A#3
- U49: footprint Custom_Electrode:Circle_2mm -> Custom_Electrode:D3_B3
- U50: footprint Custom_Electrode:Circle_2mm -> Custom_Electrode:D3_C4
- U51: footprint Custom_Electrode:Circle_2mm -> Custom_Electrode:D3_C#4
- U52: footprint Custom_Electrode:Circle_2mm -> Custom_Electrode:D3_D4
- U53: footprint Custom_Electrode:Circle_2mm -> Custom_Electrode:D3_D#4
- U54: footprint Custom_Electrode:Circle_2mm -> Custom_Electrode:D3_E4
- U55: footprint Custom_Electrode:Circle_2mm -> Custom_Electrode:D3_F4
- U56: footprint Custom_Electrode:Circle_2mm -> Custom_Electrode:D3_F#4
- U57: footprint Custom_Electrode:Circle_2mm -> Custom_Electrode:D3_G4
- U58: footprint Custom_Electrode:Circle_2mm -> Custom_Electrode:D3_G#4
- U59: footprint Custom_Electrode:Circle_2mm -> Custom_Electrode:D3_A4
- U60: footprint Custom_Electrode:Circle_2mm -> Custom_Electrode:D3_A#4
- U61: footprint Custom_Electrode:Circle_2mm -> Custom_Electrode:G3_G#3
- U62: footprint Custom_Electrode:Circle_2mm -> Custom_Electrode:G3_A3
- U63: footprint Custom_Electrode:Circle_2mm -> Custom_Electrode:G3_A#3
- U64: footprint Custom_Electrode:Circle_2mm -> Custom_Electrode:G3_B3
- U65: footprint Custom_Electrode:Circle_2mm -> Custom_Electrode:G3_C4
- U66: footprint Custom_Electrode:Circle_2mm -> Custom_Electrode:G3_C#4
- U67: footprint Custom_Electrode:Circle_2mm -> Custom_Electrode:G3_D4
- U68: footprint Custom_Electrode:Circle_2mm -> Custom_Electrode:G3_D#4
- U69: footprint Custom_Electrode:Circle_2mm -> Custom_Electrode:G3_E4
- U70: footprint Custom_Electrode:Circle_2mm -> Custom_Electrode:G3_F4
- U71: footprint Custom_Electrode:Circle_2mm -> Custom_Electrode:G3_F#4
- U72: footprint Custom_Electrode:Circle_2mm -> Custom_Electrode:G3_G4
- U73: footprint Custom_Electrode:Circle_2mm -> Custom_Electrode:G3_G#4
- U74: footprint Custom_Electrode:Circle_2mm -> Custom_Electrode:G3_A4
- U75: footprint Custom_Electrode:Circle_2mm -> Custom_Electrode:G3_A#4
- U76: footprint Custom_Electrode:Circle_2mm -> Custom_Electrode:G3_B4
- U77: footprint Custom_Electrode:Circle_2mm -> Custom_Electrode:G3_C5
- U78: footprint Custom_Electrode:Circle_2mm -> Custom_Electrode:G3_C#5
- U79: footprint Custom_Electrode:Circle_2mm -> Custom_Electrode:G3_D5
- U80: footprint Custom_Electrode:Circle_2mm -> Custom_Electrode:G3_D#5

Commit message: Added all frets on pcb
Parts:
- U100: footprint Custom_Electrode:Circle_2mm -> Custom_Electrode:B3_G5
- U101: footprint Custom_Electrode:Circle_2mm -> Custom_Electrode:E4_F4
- U102: footprint Custom_Electrode:Circle_2mm -> Custom_Electrode:E4_F#4
- U103: footprint Custom_Electrode:Circle_2mm -> Custom_Electrode:E4_G4
- U104: footprint Custom_Electrode:Circle_2mm -> Custom_Electrode:E4_G#4
- U105: footprint Custom_Electrode:Circle_2mm -> Custom_Electrode:E4_A4
- U106: footprint Custom_Electrode:Circle_2mm -> Custom_Electrode:E4_A#4
- U107: footprint Custom_Electrode:Circle_2mm -> Custom_Electrode:E4_B4
- U108: footprint Custom_Electrode:Circle_2mm -> Custom_Electrode:E4_C5
- U109: footprint Custom_Electrode:Circle_2mm -> Custom_Electrode:E4_C#5
- U110: footprint Custom_Electrode:Circle_2mm -> Custom_Electrode:E4_D5
- U111: footprint Custom_Electrode:Circle_2mm -> Custom_Electrode:E4_D#5
- U112: footprint Custom_Electrode:Circle_2mm -> Custom_Electrode:E4_E5
- U113: footprint Custom_Electrode:Circle_2mm -> Custom_Electrode:E4_F5
- U114: footprint Custom_Electrode:Circle_2mm -> Custom_Electrode:E4_F#5
- U115: footprint Custom_Electrode:Circle_2mm -> Custom_Electrode:E4_G5
- U116: footprint Custom_Electrode:Circle_2mm -> Custom_Electrode:E4_G#5
- U117: footprint Custom_Electrode:Circle_2mm -> Custom_Electrode:E4_A5
- U118: footprint Custom_Electrode:Circle_2mm -> Custom_Electrode:E4_A#5
- U119: footprint Custom_Electrode:Circle_2mm -> Custom_Electrode:E4_B5
- U120: footprint Custom_Electrode:E4_Fret20 -> Custom_Electrode:E4_C6
- U81: footprint Custom_Electrode:Circle_2mm -> Custom_Electrode:B3_C4
- U82: footprint Custom_Electrode:Circle_2mm -> Custom_Electrode:B3_C#4
- U83: footprint Custom_Electrode:Circle_2mm -> Custom_Electrode:B3_D4
- U84: footprint Custom_Electrode:Circle_2mm -> Custom_Electrode:B3_D#4
- U85: footprint Custom_Electrode:Circle_2mm -> Custom_Electrode:B3_E4
- U86: footprint Custom_Electrode:Circle_2mm -> Custom_Electrode:B3_F4
- U87: footprint Custom_Electrode:Circle_2mm -> Custom_Electrode:B3_F#4
- U88: footprint Custom_Electrode:Circle_2mm -> Custom_Electrode:B3_G4
- U89: footprint Custom_Electrode:Circle_2mm -> Custom_Electrode:B3_G#4
- U90: footprint Custom_Electrode:Circle_2mm -> Custom_Electrode:B3_A4
- U91: footprint Custom_Electrode:Circle_2mm -> Custom_Electrode:B3_A#4
- U92: footprint Custom_Electrode:Circle_2mm -> Custom_Electrode:B3_B4
- U93: footprint Custom_Electrode:Circle_2mm -> Custom_Electrode:B3_C5
- U94: footprint Custom_Electrode:Circle_2mm -> Custom_Electrode:B3_C#5
- U95: footprint Custom_Electrode:Circle_2mm -> Custom_Electrode:B3_D5
- U96: footprint Custom_Electrode:Circle_2mm -> Custom_Electrode:B3_D#5
- U97: footprint Custom_Electrode:Circle_2mm -> Custom_Electrode:B3_E5
- U98: footprint Custom_Electrode:Circle_2mm -> Custom_Electrode:B3_F5
- U99: footprint Custom_Electrode:Circle_2mm -> Custom_Electrode:B3_F#5

Commit message: Tracing is31se5100
Parts:
- removed J1, J2, J3, J4, J5, J6: Conn_01x20, Connector_PinHeader_2.54mm:PinHeader_1x20_P2.54mm_Vertical, symbol Connector_Generic:Conn_01x20
- added J?: Conn_02x04_Top_Bottom, symbol Connector_Generic:Conn_02x04_Top_Bottom
- added U121, U122, U123, U124, U125, U126, U127, U128, U129, U130, U131, U132, U133, U134, U135, U136, U137, U138: IS31SE5100-SALS2, Package_SO:SSOP-24_5.3x8.2mm_P0.65mm, symbol Custom_Sensor_Touch:IS31SE5100-SALS2
- added U139: MAX7301, Custom:MAX7301AAX, symbol Custom_Interface_Expansion:MAX7301
Connections:
- net Electrode_1: now reaches U1.1
- net Electrode_1: now also U121.6 (CAP1)
- net Electrode_10: now reaches U10.1
- net Electrode_10: now also U122.7 (CAP2)
- net Electrode_11: now reaches U11.1
- net Electrode_11: now also U122.8 (CAP3)
- net Electrode_12: now reaches U12.1
- net Electrode_12: now also U122.9 (CAP4)
- net Electrode_13: now reaches U13.1
- net Electrode_13: now also U122.11 (CAP5)
- net Electrode_14: now reaches U14.1
- net Electrode_14: now also U122.12 (CAP6)
- net Electrode_15: now reaches U15.1
- net Electrode_15: now also U122.13 (CAP7)
- net Electrode_16: now reaches U16.1
- net Electrode_16: now also U122.10 (CAP8)
- net Electrode_17: now reaches U17.1
- net Electrode_17: now also U123.6 (CAP1)
- net Electrode_18: now reaches U18.1
- net Electrode_18: now also U123.7 (CAP2)
- net Electrode_19: now reaches U19.1
- net Electrode_19: now also U123.8 (CAP3)
- net Electrode_2: now reaches U2.1
- net Electrode_2: now also U121.7 (CAP2)
- net Electrode_20: now reaches U20.1
- net Electrode_20: now also U123.9 (CAP4)
- net Electrode_3: now reaches U3.1
- net Electrode_3: now also U121.8 (CAP3)
- net Electrode_4: now reaches U4.1
- net Electrode_4: now also U121.9 (CAP4)
- net Electrode_5: now reaches U5.1
- net Electrode_5: now also U121.11 (CAP5)
- net Electrode_6: now reaches U6.1
- net Electrode_6: now also U121.12 (CAP6)
- net Electrode_7: now reaches U7.1
- net Electrode_7: now also U121.13 (CAP7)
- net Electrode_8: now reaches U8.1
- net Electrode_8: now also U121.10 (CAP8)
- net Electrode_9: now reaches U9.1
- net Electrode_9: now also U122.6 (CAP1)
- net Electrode_21: now reaches U21.1
- net Electrode_21: now also U124.6 (CAP1)
- net Electrode_30: now reaches U30.1
- net Electrode_30: now also U125.7 (CAP2)
- net Electrode_31: now reaches U31.1
- net Electrode_31: now also U125.8 (CAP3)
- net Electrode_32: now reaches U32.1
- net Electrode_32: now also U125.9 (CAP4)
- net Electrode_33: now reaches U33.1
- net Electrode_33: now also U125.11 (CAP5)
- net Electrode_34: now reaches U34.1
- net Electrode_34: now also U125.12 (CAP6)
- net Electrode_35: now reaches U35.1
- net Electrode_35: now also U125.13 (CAP7)
- net Electrode_36: now reaches U36.1
- net Electrode_36: now also U125.10 (CAP8)
- net Electrode_37: now reaches U37.1
- net Electrode_37: now also U126.6 (CAP1)
- net Electrode_38: now reaches U38.1
- net Electrode_38: now also U126.7 (CAP2)
- net Electrode_39: now reaches U39.1
- net Electrode_39: now also U126.8 (CAP3)
- net Electrode_22: now reaches U22.1
- net Electrode_22: now also U124.7 (CAP2)
- net Electrode_40: now reaches U40.1
- net Electrode_40: now also U126.9 (CAP4)
- net Electrode_23: now reaches U23.1
- net Electrode_23: now also U124.8 (CAP3)
- net Electrode_24: now reaches U24.1
- net Electrode_24: now also U124.9 (CAP4)
- net Electrode_25: now reaches U25.1
- net Electrode_25: now also U124.11 (CAP5)
- net Electrode_26: now reaches U26.1
- net Electrode_26: now also U124.12 (CAP6)
- net Electrode_27: now reaches U27.1
- net Electrode_27: now also U124.13 (CAP7)
- net Electrode_28: now reaches U28.1
- net Electrode_28: now also U124.10 (CAP8)
- net Electrode_29: now reaches U29.1
- net Electrode_29: now also U125.6 (CAP1)
- net Electrode_41: now reaches U41.1
- net Electrode_41: now also U127.6 (CAP1)
- net Electrode_50: now reaches U50.1
- net Electrode_50: now also U128.7 (CAP2)
- net Electrode_51: now reaches U51.1
- net Electrode_51: now also U128.8 (CAP3)
- net Electrode_52: now reaches U52.1
- net Electrode_52: now also U128.9 (CAP4)
- net Electrode_53: now reaches U53.1
- net Electrode_53: now also U128.11 (CAP5)
- net Electrode_54: now reaches U54.1
- net Electrode_54: now also U128.12 (CAP6)
- net Electrode_55: now reaches U55.1
- net Electrode_55: now also U128.13 (CAP7)
- net Electrode_56: now reaches U56.1
- net Electrode_56: now also U128.10 (CAP8)
- net Electrode_57: now reaches U57.1
- net Electrode_57: now also U129.6 (CAP1)
- net Electrode_58: now reaches U58.1
- net Electrode_58: now also U129.7 (CAP2)
- net Electrode_59: now reaches U59.1
- net Electrode_59: now also U129.8 (CAP3)
- net Electrode_42: now reaches U42.1
- net Electrode_42: now also U127.7 (CAP2)
- net Electrode_60: now reaches U60.1
- net Electrode_60: now also U129.9 (CAP4)
- net Electrode_43: now reaches U43.1
- net Electrode_43: now also U127.8 (CAP3)
- net Electrode_44: now reaches U44.1
- net Electrode_44: now also U127.9 (CAP4)
- net Electrode_45: now reaches U45.1
- net Electrode_45: now also U127.11 (CAP5)
- net Electrode_46: now reaches U46.1
- net Electrode_46: now also U127.12 (CAP6)
- net Electrode_47: now reaches U47.1
- net Electrode_47: now also U127.13 (CAP7)
- net Electrode_48: now reaches U48.1
- net Electrode_48: now also U127.10 (CAP8)
- net Electrode_49: now reaches U49.1
- net Electrode_49: now also U128.6 (CAP1)
- net Electrode_61: now reaches U61.1
- net Electrode_61: now also U130.6 (CAP1)
- net Electrode_70: now reaches U70.1
- net Electrode_70: now also U131.7 (CAP2)
- net Electrode_71: now reaches U71.1
- net Electrode_71: now also U131.8 (CAP3)
- net Electrode_72: now reaches U72.1
- net Electrode_72: now also U131.9 (CAP4)
- net Electrode_73: now reaches U73.1
- net Electrode_73: now also U131.11 (CAP5)
- net Electrode_74: now reaches U74.1
- net Electrode_74: now also U131.12 (CAP6)
- net Electrode_75: now reaches U75.1
- net Electrode_75: now also U131.13 (CAP7)
- net Electrode_76: now reaches U76.1
- net Electrode_76: now also U131.10 (CAP8)
- net Electrode_77: now reaches U77.1
- net Electrode_77: now also U132.6 (CAP1)
- net Electrode_78: now reaches U78.1
- net Electrode_78: now also U132.7 (CAP2)
- net Electrode_79: now reaches U79.1
- net Electrode_79: now also U132.8 (CAP3)
- net Electrode_62: now reaches U62.1
- net Electrode_62: now also U130.7 (CAP2)
- net Electrode_80: now reaches U80.1
- net Electrode_80: now also U132.9 (CAP4)
- net Electrode_63: now reaches U63.1
- net Electrode_63: now also U130.8 (CAP3)
- net Electrode_64: now reaches U64.1
- net Electrode_64: now also U130.9 (CAP4)
- net Electrode_65: now reaches U65.1
- net Electrode_65: now also U130.11 (CAP5)
- net Electrode_66: now reaches U66.1
- net Electrode_66: now also U130.12 (CAP6)
- net Electrode_67: now reaches U67.1
- net Electrode_67: now also U130.13 (CAP7)
- net Electrode_68: now reaches U68.1
- net Electrode_68: now also U130.10 (CAP8)
- net Electrode_69: now reaches U69.1
- net Electrode_69: now also U131.6 (CAP1)
- net Electrode_81: now reaches U81.1
- net Electrode_81: now also U133.6 (CAP1)
- net Electrode_90: now reaches U90.1
- net Electrode_90: now also U134.7 (CAP2)
- net Electrode_92: now reaches U92.1
- net Electrode_92: now also U134.9 (CAP4)
- net Electrode_93: now reaches U93.1
- net Electrode_93: now also U134.11 (CAP5)
- net Electrode_94: now reaches U94.1
- net Electrode_94: now also U134.12 (CAP6)
- net Electrode_95: now reaches U95.1
- net Electrode_95: now also U134.13 (CAP7)
- net Electrode_96: now reaches U96.1
- net Electrode_96: now also U134.10 (CAP8)
- net Electrode_97: now reaches U97.1
- net Electrode_97: now also U135.6 (CAP1)
- net Electrode_98: now reaches U98.1
- net Electrode_98: now also U135.7 (CAP2)
- net Electrode_99: now reaches U99.1
- net Electrode_99: now also U135.8 (CAP3)
- net Electrode_82: now reaches U82.1
- net Electrode_82: now also U133.7 (CAP2)
- net Electrode_100: now reaches U100.1
- net Electrode_100: now also U135.9 (CAP4)
- net Electrode_83: now reaches U83.1
- net Electrode_83: now also U133.8 (CAP3)
- net Electrode_84: now reaches U84.1
- net Electrode_84: now also U133.9 (CAP4)
- net Electrode_85: now reaches U85.1
- net Electrode_85: now also U133.11 (CAP5)
- net Electrode_86: now reaches U86.1
- net Electrode_86: now also U133.12 (CAP6)
- net Electrode_87: now reaches U87.1
- net Electrode_87: now also U133.13 (CAP7)
- net Electrode_88: now reaches U88.1
- net Electrode_88: now also U133.10 (CAP8)
- net Electrode_89: now reaches U89.1
- net Electrode_89: now also U134.6 (CAP1)
- net Electrode_91: now reaches U91.1
- net Electrode_91: now also U134.8 (CAP3)
- net Electrode_101: now reaches U101.1
- net Electrode_101: now also U136.6 (CAP1)
- net Electrode_110: now reaches U110.1
- net Electrode_110: now also U137.7 (CAP2)
- net Electrode_111: now reaches U111.1
- net Electrode_111: now also U137.8 (CAP3)
- net Electrode_112: now reaches U112.1
- net Electrode_112: now also U137.9 (CAP4)
- net Electrode_113: now reaches U113.1
- net Electrode_113: now also U137.11 (CAP5)
- net Electrode_114: now reaches U114.1
- net Electrode_114: now also U137.12 (CAP6)
- net Electrode_115: now reaches U115.1
- net Electrode_115: now also U137.13 (CAP7)
- net Electrode_116: now reaches U116.1
- net Electrode_116: now also U137.10 (CAP8)
- net Electrode_117: now reaches U117.1
- net Electrode_117: now also U138.6 (CAP1)
- net Electrode_118: now reaches U118.1
- net Electrode_118: now also U138.7 (CAP2)
- net Electrode_119: now reaches U119.1
- net Electrode_119: now also U138.8 (CAP3)
- net Electrode_102: now reaches U102.1
- net Electrode_102: now also U136.7 (CAP2)
- net Electrode_120: now reaches U120.1
- net Electrode_120: now also U138.9 (CAP4)
- net Electrode_103: now reaches U103.1
- net Electrode_103: now also U136.8 (CAP3)
- net Electrode_104: now reaches U104.1
- net Electrode_104: now also U136.9 (CAP4)
- net Electrode_105: now reaches U105.1
- net Electrode_105: now also U136.11 (CAP5)
- net Electrode_106: now reaches U106.1
- net Electrode_106: now also U136.12 (CAP6)
- net Electrode_107: now reaches U107.1
- net Electrode_107: now also U136.13 (CAP7)
- net Electrode_108: now reaches U108.1
- net Electrode_108: now also U136.10 (CAP8)
- net Electrode_109: now reaches U109.1
- net Electrode_109: now also U137.6 (CAP1)
- new net RELAY_1: U121.19 (OUT1), U139.32 (P4)
- new net RELAY_2: U121.20 (OUT2), U139.30 (P5)
- new net RELAY_3: U121.21 (OUT3), U139.28 (P6)
- new net RELAY_4: U121.23 (OUT4), U139.26 (P7)
- new net RELAY_5: U121.24 (OUT5), U139.5 (P8)
- new net RELAY_6: U121.1 (OUT6), U139.7 (P9)
- new net RELAY_7: U121.2 (OUT7), U139.9 (P10)
- new net RELAY_8: U121.3 (OUT8), U139.11 (P11)
- no-connect marks 0 -> 340
Other:
- moved on the sheet: U1, U10, U11, U12, U13, U14, U15, U16, U17, U18, U19, U2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
