File: capacitive_fingerboard_guitar_650/capacitive_fingerboard_guitar_650.sch (KiCad schematic (older format))
At the start: 140 parts, among them U1 Electrode, U10 Electrode, U100 Electrode, U101 Electrode, U102 Electrode, U103 Electrode, U104 Electrode, U105 Electrode, U106 Electrode, U107 Electrode, U108 Electrode, U109 Electrode, U11 Electrode, U110 Electrode, U111 Electrode, U112 Electrode, U113 Electrode, U114 Electrode, U115 Electrode, U116 Electrode, U117 Electrode, U118 Electrode, U119 Electrode, U12 Electrode, U120 Electrode, U121 IS31SE5100-SALS2, U122 IS31SE5100-SALS2, U123 IS31SE5100-SALS2, U124 IS31SE5100-SALS2, U125 IS31SE5100-SALS2, U126 IS31SE5100-SALS2, U127 IS31SE5100-SALS2, U128 IS31SE5100-SALS2, U129 IS31SE5100-SALS2, U13 Electrode, U130 IS31SE5100-SALS2, U131 IS31SE5100-SALS2, U132 IS31SE5100-SALS2, U133 IS31SE5100-SALS2, U134 IS31SE5100-SALS2, U135 IS31SE5100-SALS2, U136 IS31SE5100-SALS2, U137 IS31SE5100-SALS2, U138 IS31SE5100-SALS2, U139 MAX7301, U14 Electrode, U15 Electrode, U16 Electrode, U17 Electrode, U18 Electrode, U19 Electrode, U2 Electrode, U20 Electrode, U21 Electrode, U22 Electrode, U23 Electrode, U24 Electrode, U25 Electrode, U26 Electrode, U27 Electrode, U28 Electrode, U29 Electrode, U3 Electrode, U30 Electrode, U31 Electrode, U32 Electrode, U33 Electrode, U34 Electrode, U35 Electrode, U36 Electrode, U37 Electrode, U38 Electrode, U39 Electrode, U4 Electrode, U40 Electrode, U41 Electrode, U42 Electrode, U43 Electrode, U44 Electrode, U45 Electrode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

Commit message: Added traces for the first third
Parts:
- removed J?: Conn_02x04_Top_Bottom, symbol Connector_Generic:Conn_02x04_Top_Bottom
- removed U121, U122, U123, U124, U125, U126, U127, U128, U129, U130, U131, U132, U133, U134, U135, U136, U137, U138: IS31SE5100-SALS2, Package_SO:SSOP-24_5.3x8.2mm_P0.65mm, symbol Custom_Sensor_Touch:IS31SE5100-SALS2
- removed U139: MAX7301, Custom:MAX7301AAX, symbol Custom_Interface_Expansion:MAX7301
- added J1, J? (x5): Conn_01x08, Custom:SAMTEC_TSM-108-01-F-SV, symbol Connector_Generic:Conn_01x08
- added J11, J12, J14, J15, J17, J18, J2, J3, J5, J6, J8, J9: Conn_02x04_Top_Bottom, Connector_Harwin:Harwin_M20-7810445_2x04_P2.54mm_Vertical, symbol Connector_Generic:Conn_02x04_Top_Bottom
Connections:
- net Electrode_1: now also J1.4 (Pin_4)
- net Electrode_10: now also J2.2 (Pin_2)
- net Electrode_100: now also J15.4 (Pin_4)
- net Electrode_101: now also J?.4 (Pin_4)
- net Electrode_102: now also J?.3 (Pin_3)
- net Electrode_103: now also J?.2 (Pin_2)
- net Electrode_104: now also J?.1 (Pin_1)
- net Electrode_105: now also J?.8 (Pin_8)
- net Electrode_106: now also J?.7 (Pin_7)
- net Electrode_107: now also J?.6 (Pin_6)
- net Electrode_108: now also J?.5 (Pin_5)
- net Electrode_109: now also J17.1 (Pin_1)
- net Electrode_11: now also J2.3 (Pin_3)
- net Electrode_110: now also J17.2 (Pin_2)
- net Electrode_111: now also J17.3 (Pin_3)
- net Electrode_112: now also J17.4 (Pin_4)
- net Electrode_113: now also J17.5 (Pin_5)
- net Electrode_114: now also J17.6 (Pin_6)
- net Electrode_115: now also J17.7 (Pin_7)
- net Electrode_116: now also J17.8 (Pin_8)
- net Electrode_117: now also J18.1 (Pin_1)
- net Electrode_118: now also J18.2 (Pin_2)
- net Electrode_119: now also J18.3 (Pin_3)
- net Electrode_12: now also J2.4 (Pin_4)
- net Electrode_120: now also J18.4 (Pin_4)
- net Electrode_13: now also J2.5 (Pin_5)
- net Electrode_14: now also J2.6 (Pin_6)
- net Electrode_15: now also J2.7 (Pin_7)
- net Electrode_16: now also J2.8 (Pin_8)
- net Electrode_17: now also J3.1 (Pin_1)
- net Electrode_18: now also J3.2 (Pin_2)
- net Electrode_19: now also J3.3 (Pin_3)
- net Electrode_2: now also J1.3 (Pin_3)
- net Electrode_20: now also J3.4 (Pin_4)
- net Electrode_21: now also J?.4 (Pin_4)
- net Electrode_22: now also J?.3 (Pin_3)
- net Electrode_23: now also J?.2 (Pin_2)
- net Electrode_24: now also J?.1 (Pin_1)
- net Electrode_25: now also J?.8 (Pin_8)
- net Electrode_26: now also J?.7 (Pin_7)
- net Electrode_27: now also J?.6 (Pin_6)
- net Electrode_28: now also J?.5 (Pin_5)
- net Electrode_29: now also J5.1 (Pin_1)
- net Electrode_3: now also J1.2 (Pin_2)
- net Electrode_30: now also J5.2 (Pin_2)
- net Electrode_31: now also J5.3 (Pin_3)
- net Electrode_32: now also J5.4 (Pin_4)
- net Electrode_33: now also J5.5 (Pin_5)
- net Electrode_34: now also J5.6 (Pin_6)
- net Electrode_35: now also J5.7 (Pin_7)
- net Electrode_36: now also J5.8 (Pin_8)
- net Electrode_37: now also J6.1 (Pin_1)
- net Electrode_38: now also J6.2 (Pin_2)
- net Electrode_39: now also J6.3 (Pin_3)
- net Electrode_4: now also J1.1 (Pin_1)
- net Electrode_40: now also J6.4 (Pin_4)
- net Electrode_41: now also J?.4 (Pin_4)
- net Electrode_42: now also J?.3 (Pin_3)
- net Electrode_43: now also J?.2 (Pin_2)
- net Electrode_44: now also J?.1 (Pin_1)
- net Electrode_45: now also J?.8 (Pin_8)
- net Electrode_46: now also J?.7 (Pin_7)
- net Electrode_47: now also J?.6 (Pin_6)
- net Electrode_48: now also J?.5 (Pin_5)
- net Electrode_49: now also J8.1 (Pin_1)
- net Electrode_5: now also J1.8 (Pin_8)
- net Electrode_50: now also J8.2 (Pin_2)
- net Electrode_51: now also J8.3 (Pin_3)
- net Electrode_52: now also J8.4 (Pin_4)
- net Electrode_53: now also J8.5 (Pin_5)
- net Electrode_54: now also J8.6 (Pin_6)
- net Electrode_55: now also J8.7 (Pin_7)
- net Electrode_56: now also J8.8 (Pin_8)
- net Electrode_57: now also J9.1 (Pin_1)
- net Electrode_58: now also J9.2 (Pin_2)
- net Electrode_59: now also J9.3 (Pin_3)
- net Electrode_6: now also J1.7 (Pin_7)
- net Electrode_60: now also J9.4 (Pin_4)
- net Electrode_61: now also J?.4 (Pin_4)
- net Electrode_62: now also J?.3 (Pin_3)
- net Electrode_63: now also J?.2 (Pin_2)
- net Electrode_64: now also J?.1 (Pin_1)
- net Electrode_65: now also J?.8 (Pin_8)
- net Electrode_66: now also J?.7 (Pin_7)
- net Electrode_67: now also J?.6 (Pin_6)
- net Electrode_68: now also J?.5 (Pin_5)
- net Electrode_69: now also J11.1 (Pin_1)
- net Electrode_7: now also J1.6 (Pin_6)
- net Electrode_70: now also J11.2 (Pin_2)
- net Electrode_71: now also J11.3 (Pin_3)
- net Electrode_72: now also J11.4 (Pin_4)
- net Electrode_73: now also J11.5 (Pin_5)
- net Electrode_74: now also J11.6 (Pin_6)
- net Electrode_75: now also J11.7 (Pin_7)
- net Electrode_76: now also J11.8 (Pin_8)
- net Electrode_77: now also J12.1 (Pin_1)
- net Electrode_78: now also J12.2 (Pin_2)
- net Electrode_79: now also J12.3 (Pin_3)
- net Electrode_8: now also J1.5 (Pin_5)
- net Electrode_80: now also J12.4 (Pin_4)
- net Electrode_81: now also J?.4 (Pin_4)
- net Electrode_82: now also J?.3 (Pin_3)
- net Electrode_83: now also J?.2 (Pin_2)
- net Electrode_84: now also J?.1 (Pin_1)
- net Electrode_85: now also J?.8 (Pin_8)
- net Electrode_86: now also J?.7 (Pin_7)
- net Electrode_87: now also J?.6 (Pin_6)
- net Electrode_88: now also J?.5 (Pin_5)
- net Electrode_89: now also J14.1 (Pin_1)
- net Electrode_9: now also J2.1 (Pin_1)
- net Electrode_90: now also J14.2 (Pin_2)
- net Electrode_91: now also J14.3 (Pin_3)
- net Electrode_92: now also J14.4 (Pin_4)
- net Electrode_93: now also J14.5 (Pin_5)
- net Electrode_94: now also J14.6 (Pin_6)
- net Electrode_95: now also J14.7 (Pin_7)
- net Electrode_96: now also J14.8 (Pin_8)
- net Electrode_97: now also J15.1 (Pin_1)
- net Electrode_98: now also J15.2 (Pin_2)
- net Electrode_99: now also J15.3 (Pin_3)
- no-connect marks 340 -> 24

Commit message: Over 50% trace done
Parts:
- removed J11, J12, J14, J15, J17, J18, J2, J3, J5, J6, J8, J9: Conn_02x04_Top_Bottom, Connector_Harwin:Harwin_M20-7810445_2x04_P2.54mm_Vertical, symbol Connector_Generic:Conn_02x04_Top_Bottom
- added J11, J12, J14, J15, J17, J18, J2, J3, J5, J6, J8, J9: Conn_01x08, Custom:SAMTEC_TSM-108-01-F-SV, symbol Connector_Generic:Conn_01x08
- gave numbers to parts that had none: 5
Connections:
- net Electrode_10: now also J2.3 (Pin_3)
- net Electrode_100: now also J15.1 (Pin_1)
- net Electrode_109: now also J18.4 (Pin_4)
- net Electrode_11: now also J2.2 (Pin_2)
- net Electrode_110: now also J18.3 (Pin_3)
- net Electrode_111: now also J18.2 (Pin_2)
- net Electrode_112: now also J18.1 (Pin_1)
- net Electrode_113: now also J18.8 (Pin_8)
- net Electrode_114: now also J18.7 (Pin_7)
- net Electrode_115: now also J18.6 (Pin_6)
- net Electrode_116: now also J18.5 (Pin_5)
- net Electrode_117: now also J17.4 (Pin_4)
- net Electrode_118: now also J17.3 (Pin_3)
- net Electrode_119: now also J17.2 (Pin_2)
- net Electrode_12: now also J2.1 (Pin_1)
- net Electrode_120: now also J17.1 (Pin_1)
- net Electrode_13: now also J2.8 (Pin_8)
- net Electrode_14: now also J2.7 (Pin_7)
- net Electrode_15: now also J2.6 (Pin_6)
- net Electrode_16: now also J2.5 (Pin_5)
- net Electrode_17: now also J3.4 (Pin_4)
- net Electrode_18: now also J3.3 (Pin_3)
- net Electrode_19: now also J3.2 (Pin_2)
- net Electrode_20: now also J3.1 (Pin_1)
- net Electrode_29: now also J6.4 (Pin_4)
- net Electrode_30: now also J6.3 (Pin_3)
- net Electrode_31: now also J6.2 (Pin_2)
- net Electrode_32: now also J6.1 (Pin_1)
- net Electrode_33: now also J6.8 (Pin_8)
- net Electrode_34: now also J6.7 (Pin_7)
- net Electrode_35: now also J6.6 (Pin_6)
- net Electrode_36: now also J6.5 (Pin_5)
- net Electrode_37: now also J5.4 (Pin_4)
- net Electrode_38: now also J5.3 (Pin_3)
- net Electrode_39: now also J5.2 (Pin_2)
- net Electrode_40: now also J5.1 (Pin_1)
- net Electrode_49: now also J9.4 (Pin_4)
- net Electrode_50: now also J9.3 (Pin_3)
- net Electrode_51: now also J9.2 (Pin_2)
- net Electrode_52: now also J9.1 (Pin_1)
- net Electrode_53: now also J9.8 (Pin_8)
- net Electrode_54: now also J9.7 (Pin_7)
- net Electrode_55: now also J9.6 (Pin_6)
- net Electrode_56: now also J9.5 (Pin_5)
- net Electrode_57: now also J8.4 (Pin_4)
- net Electrode_58: now also J8.3 (Pin_3)
- net Electrode_59: now also J8.2 (Pin_2)
- net Electrode_60: now also J8.1 (Pin_1)
- net Electrode_69: now also J12.4 (Pin_4)
- net Electrode_70: now also J12.3 (Pin_3)
- net Electrode_71: now also J12.2 (Pin_2)
- net Electrode_72: now also J12.1 (Pin_1)
- net Electrode_73: now also J12.8 (Pin_8)
- net Electrode_74: now also J12.7 (Pin_7)
- net Electrode_75: now also J12.6 (Pin_6)
- net Electrode_76: now also J12.5 (Pin_5)
- net Electrode_77: now also J11.4 (Pin_4)
- net Electrode_78: now also J11.3 (Pin_3)
- net Electrode_79: now also J11.2 (Pin_2)
- net Electrode_80: now also J11.1 (Pin_1)
- net Electrode_89: now also J14.4 (Pin_4)
- net Electrode_9: now also J2.4 (Pin_4)
- net Electrode_90: now also J14.3 (Pin_3)
- net Electrode_91: now also J14.2 (Pin_2)
- net Electrode_92: now also J14.1 (Pin_1)
- net Electrode_93: now also J14.8 (Pin_8)
- net Electrode_94: now also J14.7 (Pin_7)
- net Electrode_95: now also J14.6 (Pin_6)
- net Electrode_96: now also J14.5 (Pin_5)
- net Electrode_97: now also J15.4 (Pin_4)
- net Electrode_98: now also J15.3 (Pin_3)
- net Electrode_99: now also J15.2 (Pin_2)
